Commit message: Added factory world with table and husky robot

File: src/devol_description/urdf/devol.urdf (robot description, URDF)
Before this commit: robot devol, 24 links, 23 joints
Links:
- link base_link_inertia: geometry collision mesh filename=package://ur_description/meshes/ur20/collision/base.stl; visual mesh filename=package://ur_description/meshes/ur20/visual/base.dae
- link forearm_link: mass 4.27 -> 7.879; geometry collision mesh filename=package://ur_description/meshes/ur20/collision/forearm.stl; visual mesh filename=package://ur_description/meshes/ur20/visual/forearm.dae
- link shoulder_link: mass 7.1 -> 16.343; geometry collision mesh filename=package://ur_description/meshes/ur20/collision/shoulder.stl; visual mesh filename=package://ur_description/meshes/ur20/visual/shoulder.dae
- link upper_arm_link: mass 12.7 -> 29.632; geometry collision mesh filename=package://ur_description/meshes/ur20/collision/upperarm.stl; visual mesh filename=package://ur_description/meshes/ur20/visual/upperarm.dae
- link wrist_1_link: mass 2.0 -> 3.054; geometry collision mesh filename=package://ur_description/meshes/ur20/collision/wrist1.stl; visual mesh filename=package://ur_description/meshes/ur20/visual/wrist1.dae
- link wrist_2_link: mass 2.0 -> 3.126; geometry collision mesh filename=package://ur_description/meshes/ur20/collision/wrist2.stl; visual mesh filename=package://ur_description/meshes/ur20/visual/wrist2.dae
- link wrist_3_link: mass 0.365 -> 0.926; geometry collision mesh filename=package://ur_description/meshes/ur20/collision/wrist3.stl; visual mesh filename=package://ur_description/meshes/ur20/visual/wrist3.dae
Joints:
- joint elbow_joint: limit lower=-3.141592653589793 upper=3.141592653589793 effort=150.0 velocity=3.141592653589793 -> lower=-3.141592653589793 upper=3.141592653589793 effort=433.0 velocity=2.6179938779914944; origin xyz=-0.612 0 0 rpy=0 0 0 -> xyz=-0.862 0 0 rpy=0 0 0
- joint shoulder_lift_joint: limit lower=-6.283185307179586 upper=6.283185307179586 effort=330.0 velocity=2.0943951023931953 -> lower=-6.283185307179586 upper=6.283185307179586 effort=738.0 velocity=2.0943951023931953
- joint shoulder_pan_joint: limit lower=-6.283185307179586 upper=6.283185307179586 effort=330.0 velocity=2.0943951023931953 -> lower=-6.283185307179586 upper=6.283185307179586 effort=738.0 velocity=2.0943951023931953; origin xyz=0 0 0.1273 rpy=0 0 0 -> xyz=0 0 0.2363 rpy=0 0 0
- joint wrist_1_joint: limit lower=-6.283185307179586 upper=6.283185307179586 effort=56.0 velocity=3.141592653589793 -> lower=-6.283185307179586 upper=6.283185307179586 effort=107.0 velocity=3.6651914291880923; origin xyz=-0.5723 0 0.163941 rpy=0 0 0 -> xyz=-0.7287 0 0.201 rpy=0 0 0
- joint wrist_2_joint: limit lower=-6.283185307179586 upper=6.283185307179586 effort=56.0 velocity=3.141592653589793 -> lower=-6.283185307179586 upper=6.283185307179586 effort=107.0 velocity=3.6651914291880923; origin xyz=0 -0.1157 -2.373046667922381e-11 rpy=1.570796327 0 0 -> xyz=0 -0.1593 -3.267297616249225e-11 rpy=1.570796327 0 0
- joint wrist_3_joint: limit lower=-6.283185307179586 upper=6.283185307179586 effort=56.0 velocity=3.141592653589793 -> lower=-6.283185307179586 upper=6.283185307179586 effort=107.0 velocity=3.6651914291880923; origin xyz=0 0.0922 -1.891053610911353e-11 rpy=1.570796326589793 3.141592653589793 3.141592653589793 -> xyz=0 0.1543 -3.1647459019915597e-11 rpy=1.570796326589793 3.141592653589793 3.141592653589793

File: src/devol_description/urdf/devol.urdf.xacro (robot description, xacro)
@@ -9,5 +9,5 @@
   <!-- possible 'ur_type' values: ur3, ur3e, ur5, ur5e, ur10, ur10e, ur16e, ur20, ur30 -->
   <!-- the default value should raise an error in case this was called without defining the type -->
-  <xacro:arg name="ur_type" default="ur10"/>
+  <xacro:arg name="ur_type" default="ur20"/>
   <!-- parameters -->
   <xacro:arg name="name" default="devol"/>
@@ -31,5 +31,5 @@
   <xacro:arg name="force_abs_paths" default="false" />
   <!-- initial position for simulations (Mock Hardware, Gazebo, Ignition) -->
-  <xacro:arg name="initial_positions_file" default="$(find ur_description)/config/initial_positions.yaml"/>
+  <xacro:arg name="initial_positions_file" default="$(find devol_description)/config/initial_positions.yaml"/>
   <!-- convert to property to use substitution in function -->
   <xacro:property name="initial_positions_file" default="$(arg initial_positions_file)"/>
