Commit message: Created bridge. Holding off on merging into main

File: src/devol_description/urdf/devol.urdf.xacro (robot description, xacro)
@@ -1,16 +1,7 @@
 <?xml version="1.0"?>
 <robot xmlns:xacro="http://wiki.ros.org/xacro" name="devol">
-  <!-- import macros -->
-  <xacro:include filename="$(find ur_description)/urdf/ur_macro.xacro"/>
-  <xacro:include filename="$(find ur_robot_driver)/urdf/ur.ros2_control.xacro"/>
-  <xacro:include filename="$(find robotiq_description)/urdf/robotiq_2f_85_macro.urdf.xacro"/>
-  <xacro:include filename="$(find robotiq_description)/urdf/robotiq_gripper.ros2_control.xacro"/>
-  <xacro:include filename="$(find robotiq_description)/urdf/ur_to_robotiq_adapter.urdf.xacro"/>
-  <!-- possible 'ur_type' values: ur3, ur3e, ur5, ur5e, ur10, ur10e, ur16e, ur20, ur30 -->
-  <!-- the default value should raise an error in case this was called without defining the type -->
-  <xacro:arg name="ur_type" default="ur20"/>
-  <!-- parameters -->
   <xacro:arg name="name" default="devol"/>
   <xacro:arg name="tf_prefix" default="" />
+  <xacro:arg name="ur_type" default="ur20"/>
   <xacro:arg name="joint_limit_params" default="$(find ur_description)/config/$(arg ur_type)/joint_limits.yaml"/>
   <xacro:arg name="kinematics_params" default="$(find ur_description)/config/$(arg ur_type)/default_kinematics.yaml"/>
@@ -21,58 +12,48 @@
   <xacro:arg name="safety_pos_margin" default="0.15"/>
   <xacro:arg name="safety_k_position" default="20"/>
-  <xacro:arg name="use_mock_hardware" default="true" />
-  <xacro:arg name="mock_sensor_commands" default="true" />
+  <xacro:arg name="use_mock_hardware" default="false" />
+  <xacro:arg name="mock_sensor_commands" default="false" />
   <xacro:arg name="robot_ip" default="yyy.yyy.yyy.yyy" />
   <xacro:arg name="script_filename" default="None" />
   <xacro:arg name="input_recipe_filename" default="None" />
   <xacro:arg name="output_recipe_filename" default="None" />
-  <!--When using gazebo simulations absolute paths are necessary.-->
-  <xacro:arg name="force_abs_paths" default="false" />
+  <xacro:arg name="use_gazebo" default="true" />
   <!-- initial position for simulations (Mock Hardware, Gazebo, Ignition) -->
   <xacro:arg name="initial_positions_file" default="$(find devol_description)/config/initial_positions.yaml"/>
   <!-- convert to property to use substitution in function -->
   <xacro:property name="initial_positions_file" default="$(arg initial_positions_file)"/>
-  <!-- arm -->
+  <!-- Import devol macro -->
+  <xacro:include filename="$(find devol_description)/urdf/devol_macro.urdf.xacro"/>
+  <!-- ros2_control description -->
+  <xacro:include filename="$(find devol_description)/urdf/devol.ros2_control.xacro"/>
   <link name="world" />
-  <xacro:ur_robot
-      name="$(arg name)"
-      tf_prefix="$(arg tf_prefix)"
-      parent="world"
-      joint_limits_parameters_file="$(arg joint_limit_params)"
-      kinematics_parameters_file="$(arg kinematics_params)"
-      physical_parameters_file="$(arg physical_params)"
-      visual_parameters_file="$(arg visual_params)"
-      safety_limits="$(arg safety_limits)"
-      safety_pos_margin="$(arg safety_pos_margin)"
-      safety_k_position="$(arg safety_k_position)"
-      force_abs_paths="$(arg force_abs_paths)"
-      >
-      <origin xyz="0 0 0" rpy="0 0 0" />          <!-- position robot in the world -->
-  </xacro:ur_robot>
-  <!-- ros2 control instance -->
-  <xacro:ur_ros2_control
-      name="$(arg name)"
-      tf_prefix="$(arg tf_prefix)"
-      kinematics_parameters_file="$(arg kinematics_params)"
-      robot_ip="$(arg robot_ip)"
-      script_filename="$(arg script_filename)"
-      input_recipe_filename="$(arg input_recipe_filename)"
-      output_recipe_filename="$(arg output_recipe_filename)"
-      use_mock_hardware="$(arg use_mock_hardware)"
-      mock_sensor_commands="$(arg mock_sensor_commands)"
-      initial_positions="${xacro.load_yaml((initial_positions_file))}"
-  />
-  <xacro:ur_to_robotiq
-    prefix="$(arg tf_prefix)"
-    connected_to="$(arg tf_prefix)tool0"
-  />
-  <xacro:robotiq_gripper
-      name="RobotiqGripperHardwareInterface"
-      parent="$(arg tf_prefix)gripper_mount_link"
-      prefix="$(arg tf_prefix)"
-      use_fake_hardware="true"
-      fake_sensor_commands="true"
-  >
+  <xacro:devol
+    parent="world"
+    name="$(arg name)"
+    tf_prefix="$(arg tf_prefix)"
+    ur_type="$(arg ur_type)"
+    joint_limit_params="$(arg joint_limit_params)"
+    kinematics_params="$(arg kinematics_params)"
+    physical_params="$(arg physical_params)"
+    visual_params="$(arg visual_params)"
+    transmission_hw_interface="$(arg transmission_hw_interface)"
+    safety_limits="$(arg safety_limits)"
+    safety_pos_margin="$(arg safety_pos_margin)"
+    safety_k_position="$(arg safety_k_position)"
+    use_mock_hardware="$(arg use_mock_hardware)"
+    mock_sensor_commands="$(arg mock_sensor_commands)"
+    robot_ip="$(arg robot_ip)"
+    script_filename="$(arg script_filename)"
+    input_recipe_filename="$(arg input_recipe_filename)"
+    output_recipe_filename="$(arg output_recipe_filename)"
+    initial_positions="${xacro.load_yaml((initial_positions_file))}"
+    use_gazebo="$(arg use_gazebo)"
+    >
     <origin xyz="0 0 0" rpy="0 0 0"/>
-  </xacro:robotiq_gripper>
+  </xacro:devol>
+  <xacro:devol_ros2_control name="Devol" prefix="$(arg tf_prefix)" use_gazebo="$(arg use_gazebo)"/>
+  <xacro:if value="$(arg use_gazebo)">
+    <xacro:include filename="$(find devol_description)/urdf/devol.gazebo.xacro"/>
+    <xacro:devol_gazebo/>
+  </xacro:if>
 </robot>

File: src/devol_moveit_config/config/devol.ros2_control.xacro (robot description, xacro)
@@ -5,5 +5,5 @@
             <hardware>
                 <!-- By default, set up controllers for simulation. This won't work on real hardware -->
-                <plugin>mock_components/GenericSystem</plugin>
+                <plugin>gz_ros2_control/GazeboSimSystem</plugin>
             </hardware>
             <joint name="shoulder_pan_joint">

File: src/devol_moveit_config/config/devol.urdf.xacro (robot description, xacro)
@@ -1,5 +1,5 @@
 <?xml version="1.0"?>
 <robot xmlns:xacro="http://www.ros.org/wiki/xacro" name="devol">
-    <xacro:arg name="initial_positions_file" default="/home/jakeadelic/programming/devol/src/devol_moveit_config/config/initial_positions.yaml" />
+    <xacro:arg name="initial_positions_file" default="$(find devol_moveit_config)/config/initial_positions.yaml" />
     <!-- Import devol urdf file -->
     <xacro:include filename="$(find devol_description)/urdf/devol.urdf.xacro" />
