Commit message: Cleaned up docker files.

File: src/devol_description/urdf/devol.gazebo.xacro (robot description, xacro)
@@ -12,6 +12,6 @@
       </plugin>
       <plugin
-        filename="libignition-gazebo-detachable-joint-system.so"
-        name="ignition::gazebo::systems::DetachableJoint">
+        filename="libgz-sim-detachable-joint-system.so"
+        name="gz::sim::systems::DetachableJoint">
         <parent_link>wrist_3_link</parent_link>
         <child_link>target_block</child_link>

File: src/devol_description/urdf/devol.ros2_control.xacro (robot description, xacro)
@@ -12,5 +12,5 @@
                 <xacro:unless value="${use_gazebo}">
                     <!-- Use Mock Hardware for real hardware -->
-                    <plugin>gz_ros2_control/MockHardware</plugin>
+                    <plugin>mock_components/GenericSystem</plugin>
                 </xacro:unless>
             </hardware>

File: src/devol_description/urdf/devol.urdf.xacro (robot description, xacro)
@@ -52,5 +52,5 @@
     <origin xyz="0 0 0" rpy="0 0 0"/>
   </xacro:devol>
-  <xacro:devol_ros2_control name="Devol" prefix="$(arg tf_prefix)" use_gazebo="$(arg use_gazebo)"/>
+  <xacro:devol_ros2_control name="devol_ros2_control" prefix="$(arg tf_prefix)" use_gazebo="$(arg use_gazebo)"/>
   <xacro:if value="$(arg use_gazebo)">
     <xacro:include filename="$(find devol_description)/urdf/devol.gazebo.xacro"/>

File: src/devol_moveit_config/config/devol.ros2_control.xacro (robot description, xacro)
@@ -1,14 +1,22 @@
 <?xml version="1.0"?>
 <robot xmlns:xacro="http://www.ros.org/wiki/xacro">
-    <xacro:macro name="devol_ros2_control" params="name">
+    <xacro:include filename="$(find ur_robot_driver)/urdf/ur.ros2_control.xacro"/>
+    <xacro:include filename="$(find robotiq_description)/urdf/robotiq_gripper.ros2_control.xacro"/>
+    <xacro:macro name="devol_ros2_control" params="name prefix use_gazebo:=^|false">
         <ros2_control name="${name}" type="system">
             <hardware>
-                <!-- By default, set up controllers for simulation. This won't work on real hardware -->
-                <plugin>gz_ros2_control/GazeboSimSystem</plugin>
+                <xacro:if value="${use_gazebo}">
+                    <!-- Use Gazebo plugin for simulation -->
+                    <plugin>gz_ros2_control/GazeboSimSystem</plugin>
+                </xacro:if>
+                <xacro:unless value="${use_gazebo}">
+                    <!-- Use Mock Hardware for real hardware -->
+                    <plugin>mock_components/GenericSystem</plugin>
+                </xacro:unless>
             </hardware>
             <joint name="shoulder_pan_joint">
                 <command_interface name="position"/>
                 <state_interface name="position">
-                  <param name="initial_value">0.0</param>
+                  <param name="initial_value">3.14159</param>
                 </state_interface>
                 <state_interface name="velocity"/>

File: src/devol_moveit_config/config/devol.urdf.xacro (robot description, xacro)
@@ -1,9 +1,8 @@
 <?xml version="1.0"?>
 <robot xmlns:xacro="http://www.ros.org/wiki/xacro" name="devol">
-    <xacro:arg name="initial_positions_file" default="$(find devol_moveit_config)/config/initial_positions.yaml" />
     <!-- Import devol urdf file -->
     <xacro:include filename="$(find devol_description)/urdf/devol.urdf.xacro" />
     <!-- Import control_xacro -->
     <xacro:include filename="$(find devol_moveit_config)/config/devol.ros2_control.xacro" />
-    <xacro:devol_ros2_control name="FakeSystem"/>
+    <xacro:devol_ros2_control prefix="fake" name="FakeSystem"/>
 </robot>

Commit message: added intel realsense D405 camera to robot's end effector

File: src/devol_description/urdf/devol.gazebo.xacro (robot description, xacro)
@@ -22,4 +22,50 @@
       </plugin>
     </gazebo>
+    <!-- Camera -->
+    <gazebo reference="camera_color_frame">
+      <sensor type="camera" name="realsense_d405_camera">
+        <pose relative_to="camera_color_frame">0 0 0 3.14159 0 0</pose>
+        <topic>camera/image_raw</topic>
+        <camera>
+          <camera_info_topic>camera/camera_info</camera_info_topic>
+          <horizontal_fov>1.518</horizontal_fov>
+          <image>
+            <width>1280</width>
+            <height>720</height>
+            <format>R8G8B8</format>
+          </image>
+          <clip>
+            <near>0.1</near>
+            <far>5.0</far>
+          </clip>
+        </camera>
+        <always_on>1</always_on>
+        <visualize>1</visualize>
+        <update_rate>30</update_rate>
+      </sensor>
+    </gazebo>
+    <!-- Depth Camera  -->
+    <gazebo reference="camera_depth_frame">
+      <sensor type="depth_camera" name="realsense_d405_depth_camera">
+        <topic>depth/image_raw</topic>
+        <pose relative_to="camera_color_frame">0 0 0 3.14159 0 0</pose>
+        <camera>
+          <camera_info_topic>depth/camera_info</camera_info_topic>
+          <horizontal_fov>1.518</horizontal_fov>
+          <image>
+            <width>1280</width>
+            <height>720</height>
+            <format>L16</format>
+          </image>
+          <clip>
+            <near>0.1</near>
+            <far>5.0</far>
+          </clip>
+        </camera>
+        <always_on>true</always_on>
+        <visualize>1</visualize>
+        <update_rate>30</update_rate>
+      </sensor>
+    </gazebo>
   </xacro:macro>
 </robot>

File: src/devol_description/urdf/devol_macro.urdf.xacro (robot description, xacro)
@@ -5,4 +5,5 @@
     <xacro:include filename="$(find robotiq_description)/urdf/robotiq_2f_85_macro.urdf.xacro"/>
     <xacro:include filename="$(find robotiq_description)/urdf/ur_to_robotiq_adapter.urdf.xacro"/>
+    <xacro:include filename= "$(find realsense2_description)/urdf/_d405.urdf.xacro"/>
     <xacro:macro name="devol" params="
         parent
@@ -50,4 +51,7 @@
             connected_to="${tf_prefix}tool0"
         />
+        <xacro:sensor_d405 parent="${tf_prefix}gripper_mount_link" use_nominal_extrinsics="true">
+            <origin xyz="0 0.08 0" rpy="0 -1.570795 1.570795"/>
+        </xacro:sensor_d405>
         <xacro:robotiq_gripper
             name="RobotiqGripperHardwareInterface"

Commit message: Working diff drive system. Need to implement moveit and rviz for devol drive

File: src/devol_description/urdf/devol.gazebo.xacro (robot description, xacro)
@@ -5,5 +5,5 @@
 -->
 <robot xmlns:xacro="http://ros.org/wiki/xacro">
-  <xacro:macro name="devol_gazebo">
+  <xacro:macro name="devol_gazebo" params="tf_prefix">
     <!-- ros_control plugin -->
     <gazebo>
@@ -11,8 +11,8 @@
         <parameters>$(find devol_description)/config/ros2_controllers.yaml</parameters>
       </plugin>
-      <plugin
+      <!-- <plugin
         filename="libgz-sim-detachable-joint-system.so"
         name="gz::sim::systems::DetachableJoint">
-        <parent_link>wrist_3_link</parent_link>
+        <parent_link>${tf_prefix}wrist_3_link</parent_link>
         <child_link>target_block</child_link>
         <child_model>target_block</child_model>
@@ -20,13 +20,13 @@
         <attach_topic>/devol_attach/attach</attach_topic>
         <detach_topic>/devol_attach/detach</detach_topic>
-      </plugin>
+      </plugin> -->
     </gazebo>
     <!-- Camera -->
     <gazebo reference="camera_color_frame">
-      <sensor type="camera" name="realsense_d405_camera">
+      <sensor type="camera" name="${tf_prefix}realsense_d405_camera">
         <pose relative_to="camera_color_frame">0 0 0 3.14159 0 0</pose>
-        <topic>camera/image_raw</topic>
+        <topic>/model/${tf_prefix}devol/color_raw</topic>
         <camera>
-          <camera_info_topic>camera/camera_info</camera_info_topic>
+          <camera_info_topic>/model/${tf_prefix}devol/color_info</camera_info_topic>
           <horizontal_fov>1.518</horizontal_fov>
           <image>
@@ -47,9 +47,9 @@
     <!-- Depth Camera  -->
     <gazebo reference="camera_depth_frame">
-      <sensor type="depth_camera" name="realsense_d405_depth_camera">
-        <topic>depth/image_raw</topic>
+      <sensor type="depth_camera" name="${tf_prefix}realsense_d405_depth_camera">
+        <topic>/model/${tf_prefix}devol/depth_raw</topic>
         <pose relative_to="camera_color_frame">0 0 0 3.14159 0 0</pose>
         <camera>
-          <camera_info_topic>depth/camera_info</camera_info_topic>
+          <camera_info_topic>/model/${tf_prefix}devol/depth_info</camera_info_topic>
           <horizontal_fov>1.518</horizontal_fov>
           <image>

File: src/devol_description/urdf/devol.ros2_control.xacro (robot description, xacro)
@@ -64,4 +64,9 @@
                 <state_interface name="velocity"/>
             </joint>
+            <joint name="robotiq_85_right_knuckle_joint" />
+            <joint name="robotiq_85_left_inner_knuckle_joint" />
+            <joint name="robotiq_85_right_inner_knuckle_joint" />
+            <joint name="robotiq_85_left_finger_tip_joint" />
+            <joint name="robotiq_85_right_finger_tip_joint" />
         </ros2_control>
     </xacro:macro>

File: src/devol_description/urdf/devol.urdf.xacro (robot description, xacro)
@@ -55,5 +55,7 @@
   <xacro:if value="$(arg use_gazebo)">
     <xacro:include filename="$(find devol_description)/urdf/devol.gazebo.xacro"/>
-    <xacro:devol_gazebo/>
+    <xacro:devol_gazebo
+      tf_prefix="$(arg tf_prefix)"
+      />
   </xacro:if>
 </robot>

File: src/devol_description/urdf/devol_macro.urdf.xacro (robot description, xacro)
@@ -27,6 +27,6 @@
         initial_positions
         *origin
-        use_gazebo:=false
-        force_abs_paths:=true
+        use_gazebo
+        force_abs_paths
     ">
         <!-- arm -->
@@ -58,6 +58,5 @@
             parent="${tf_prefix}gripper_mount_link"
             prefix="${tf_prefix}"
-            use_fake_hardware="true"
-            fake_sensor_commands="false"
+            include_ros2_control="${not use_gazebo}"
         >
             <origin xyz="0 0 0" rpy="0 0 0"/>
@@ -78,8 +77,4 @@
                 initial_positions="${initial_positions}"
             />
-            <!-- <xacro:robotiq_gripper_ros2_control
-                name="RobotiqGripperHardwareInterface"
-                prefix="${tf_prefix}"
-            /> -->
         </xacro:unless>
     </xacro:macro>
