Commit message: working dual devol demo

File: src/devol_description/urdf/devol.gazebo.xacro (robot description, xacro)
@@ -8,14 +8,14 @@
     <!-- ros_control plugin -->
     <gazebo>
-      <plugin filename="gz_ros2_control-system" name="gz_ros2_control::GazeboSimROS2ControlPlugin">
+      <!-- <plugin filename="gz_ros2_control-system" name="gz_ros2_control::GazeboSimROS2ControlPlugin">
         <parameters>$(find devol_description)/config/ros2_controllers.yaml</parameters>
-      </plugin>
+      </plugin> -->
       <plugin
         filename="libgz-sim-detachable-joint-system.so"
         name="gz::sim::systems::DetachableJoint">
         <parent_link>${tf_prefix}wrist_3_link</parent_link>
-        <child_link>target_block</child_link>
-        <child_model>target_block</child_model>
-        <child_model_link>target_block</child_model_link>
+        <child_link>target_block_0</child_link>
+        <child_model>target_block_0</child_model>
+        <child_model_link>target_block_0</child_model_link>
         <attach_topic>/${tf_prefix}devol_attach/attach</attach_topic>
         <detach_topic>/${tf_prefix}devol_attach/detach</detach_topic>
@@ -23,7 +23,7 @@
     </gazebo>
     <!-- Camera -->
-    <gazebo reference="camera_color_frame">
+    <gazebo reference="${tf_prefix}_camera_color_frame">
       <sensor type="camera" name="${tf_prefix}realsense_d405_camera">
-        <pose relative_to="camera_color_frame">0 0 0 3.14159 0 0</pose>
+        <pose relative_to="${tf_prefix}_camera_color_frame">0 0 0 3.14159 0 0</pose>
         <topic>/model/${tf_prefix}devol/color_raw</topic>
         <camera>
@@ -46,8 +46,8 @@
     </gazebo>
     <!-- Depth Camera  -->
-    <gazebo reference="camera_depth_frame">
+    <gazebo reference="${tf_prefix}_camera_depth_frame">
       <sensor type="depth_camera" name="${tf_prefix}realsense_d405_depth_camera">
         <topic>/model/${tf_prefix}devol/depth_raw</topic>
-        <pose relative_to="camera_color_frame">0 0 0 3.14159 0 0</pose>
+        <pose relative_to="${tf_prefix}_camera_color_frame">0 0 0 3.14159 0 0</pose>
         <camera>
           <camera_info_topic>/model/${tf_prefix}devol/depth_info</camera_info_topic>

File: src/devol_description/urdf/devol.ros2_control.xacro (robot description, xacro)
@@ -3,5 +3,5 @@
     <xacro:include filename="$(find ur_robot_driver)/urdf/ur.ros2_control.xacro"/>
     <xacro:include filename="$(find robotiq_description)/urdf/robotiq_gripper.ros2_control.xacro"/>
-    <xacro:macro name="devol_ros2_control" params="name prefix use_gazebo:=^|false">
+    <xacro:macro name="devol_ros2_control" params="name tf_prefix use_gazebo:=^|false">
         <ros2_control name="${name}" type="system">
             <hardware>
@@ -15,5 +15,5 @@
                 </xacro:unless>
             </hardware>
-            <joint name="shoulder_pan_joint">
+            <joint name="${tf_prefix}shoulder_pan_joint">
                 <command_interface name="position"/>
                 <state_interface name="position">
@@ -22,5 +22,5 @@
                 <state_interface name="velocity"/>
             </joint>
-            <joint name="shoulder_lift_joint">
+            <joint name="${tf_prefix}shoulder_lift_joint">
                 <command_interface name="position"/>
                 <state_interface name="position">
@@ -29,5 +29,5 @@
                 <state_interface name="velocity"/>
             </joint>
-            <joint name="elbow_joint">
+            <joint name="${tf_prefix}elbow_joint">
                 <command_interface name="position"/>
                 <state_interface name="position">
@@ -36,5 +36,5 @@
                 <state_interface name="velocity"/>
             </joint>
-            <joint name="wrist_1_joint">
+            <joint name="${tf_prefix}wrist_1_joint">
                 <command_interface name="position"/>
                 <state_interface name="position">
@@ -43,5 +43,5 @@
                 <state_interface name="velocity"/>
             </joint>
-            <joint name="wrist_2_joint">
+            <joint name="${tf_prefix}wrist_2_joint">
                 <command_interface name="position"/>
                 <state_interface name="position">
@@ -50,5 +50,5 @@
                 <state_interface name="velocity"/>
             </joint>
-            <joint name="wrist_3_joint">
+            <joint name="${tf_prefix}wrist_3_joint">
                 <command_interface name="position"/>
                 <state_interface name="position">
@@ -57,5 +57,5 @@
                 <state_interface name="velocity"/>
             </joint>
-            <joint name="robotiq_85_left_knuckle_joint">
+            <joint name="${tf_prefix}robotiq_85_left_knuckle_joint">
                 <command_interface name="position"/>
                 <state_interface name="position">
@@ -64,9 +64,9 @@
                 <state_interface name="velocity"/>
             </joint>
-            <joint name="robotiq_85_right_knuckle_joint" />
-            <joint name="robotiq_85_left_inner_knuckle_joint" />
-            <joint name="robotiq_85_right_inner_knuckle_joint" />
-            <joint name="robotiq_85_left_finger_tip_joint" />
-            <joint name="robotiq_85_right_finger_tip_joint" />
+            <joint name="${tf_prefix}robotiq_85_right_knuckle_joint" />
+            <joint name="${tf_prefix}robotiq_85_left_inner_knuckle_joint" />
+            <joint name="${tf_prefix}robotiq_85_right_inner_knuckle_joint" />
+            <joint name="${tf_prefix}robotiq_85_left_finger_tip_joint" />
+            <joint name="${tf_prefix}robotiq_85_right_finger_tip_joint" />
         </ros2_control>
     </xacro:macro>

File: src/devol_description/urdf/devol.urdf.xacro (robot description, xacro)
@@ -53,5 +53,5 @@
     <origin xyz="0 0 0" rpy="0 0 0"/>
   </xacro:devol>
-  <xacro:devol_ros2_control name="devol_ros2_control" prefix="$(arg tf_prefix)" use_gazebo="$(arg use_gazebo)"/>
+  <xacro:devol_ros2_control name="devol_ros2_control" tf_prefix="$(arg tf_prefix)" use_gazebo="$(arg use_gazebo)"/>
   <xacro:if value="$(arg use_gazebo)">
     <xacro:include filename="$(find devol_description)/urdf/devol.gazebo.xacro"/>

File: src/devol_description/urdf/devol_macro.urdf.xacro (robot description, xacro)
@@ -51,5 +51,5 @@
             connected_to="${tf_prefix}tool0"
         />
-        <xacro:sensor_d405 parent="${tf_prefix}gripper_mount_link" use_nominal_extrinsics="true">
+        <xacro:sensor_d405 parent="${tf_prefix}gripper_mount_link" name="${tf_prefix}_camera" use_nominal_extrinsics="true">
             <origin xyz="0 0.08 0" rpy="0 -1.570795 1.570795"/>
         </xacro:sensor_d405>
@@ -58,9 +58,9 @@
             parent="${tf_prefix}gripper_mount_link"
             prefix="${tf_prefix}"
-            include_ros2_control="${not use_gazebo}"
+            include_ros2_control="${not use_gazebo and not use_mock_hardware}"
         >
             <origin xyz="0 0 0" rpy="0 0 0"/>
         </xacro:robotiq_gripper>
-        <xacro:unless value="${use_gazebo}">
+        <xacro:unless value="${use_gazebo or use_mock_hardware}">
             <xacro:include filename="$(find ur_robot_driver)/urdf/ur.ros2_control.xacro"/>
             <xacro:include filename="$(find robotiq_description)/urdf/robotiq_gripper.ros2_control.xacro"/>

File: src/devol_drive_description/urdf/devol_drive.gazebo.xacro (robot description, xacro)
@@ -8,12 +8,12 @@
     <!-- Gazebo Parameters -->
     <xacro:include filename="$(find diff_drive_description)/urdf/diff_drive.gazebo.xacro"/>
+    <xacro:include filename="$(find devol_description)/urdf/devol.gazebo.xacro"/>
     <xacro:diff_drive_gazebo
-        wheel_separation="${(wheel_separation)}"
-        wheel_radius="$(arg wheel_radius)"
-        max_linear_acceleration="$(arg max_linear_acceleration)"
-        tf_prefix="$(arg tf_prefix)"/>
-    <xacro:include filename="$(find devol_description)/urdf/devol.gazebo.xacro"/>
+        wheel_separation="${wheel_separation}"
+        wheel_radius="${wheel_radius}"
+        max_linear_acceleration="${max_linear_acceleration}"
+        tf_prefix="${tf_prefix}"/>
     <xacro:devol_gazebo
-      tf_prefix="$(arg tf_prefix)"
+      tf_prefix="${tf_prefix}"
       />
   </xacro:macro>

File: src/devol_drive_description/urdf/devol_drive.urdf.xacro (robot description, xacro)
@@ -5,5 +5,5 @@
     <xacro:include filename="$(find devol_drive_description)/urdf/devol_drive_macro.urdf.xacro"/>
     <!-- ros2_control description -->
-    <xacro:include filename="$(find devol_description)/urdf/devol.ros2_control.xacro"/>
+    <xacro:include filename="$(find devol_drive_description)/urdf/devol_drive.ros2_control.xacro"/>
     <!-- Robot Parameters -->
     <xacro:arg name="parent" default="empty"/>  <!-- Set this to world for rviz and others -->
@@ -78,5 +78,5 @@
         <origin xyz="0 0 0" rpy="0 0 0"/>
     </xacro:devol_drive>
-    <xacro:devol_ros2_control name="devol_ros2_control" prefix="$(arg tf_prefix)" use_gazebo="$(arg use_gazebo)"/>
+    <xacro:devol_drive_ros2_control tf_prefix="$(arg tf_prefix)" use_gazebo="$(arg use_gazebo)"/>
     <xacro:if value="$(arg use_gazebo)">
         <xacro:include filename="$(find devol_drive_description)/urdf/devol_drive.gazebo.xacro"/>

File: src/devol_drive_description/urdf/devol_drive_macro.urdf.xacro (robot description, xacro)
@@ -41,39 +41,39 @@
         <xacro:property name="caster_offset" value="${body_length/2 - caster_radius}"/>
         <xacro:diff_drive
-            parent="$(arg parent)"
-            tf_prefix="$(arg tf_prefix)"
-            body_length="$(arg body_length)"
-            body_width="$(arg body_width)"
-            body_height="$(arg body_height)"
-            body_density="$(arg body_density)"
-            wheel_radius="$(arg wheel_radius)"
-            wheel_width="$(arg wheel_width)"
-            wheel_density="$(arg wheel_density)"
-            caster_radius="$(arg caster_radius)"
-            caster_density="$(arg caster_density)"
-            max_linear_acceleration="$(arg max_linear_acceleration)"
+            parent="${parent}"
+            tf_prefix="${tf_prefix}"
+            body_length="${body_length}"
+            body_width="${body_width}"
+            body_height="${body_height}"
+            body_density="${body_density}"
+            wheel_radius="${wheel_radius}"
+            wheel_width="${wheel_width}"
+            wheel_density="${wheel_density}"
+            caster_radius="${caster_radius}"
+            caster_density="${caster_density}"
+            max_linear_acceleration="${max_linear_acceleration}"
         />
         <xacro:devol
-            parent="$(arg tf_prefix)body_link"
-            name="$(arg name)"
-            tf_prefix="$(arg tf_prefix)"
-            ur_type="$(arg ur_type)"
-            joint_limit_params="$(arg joint_limit_params)"
-            kinematics_params="$(arg kinematics_params)"
-            physical_params="$(arg physical_params)"
-            visual_params="$(arg visual_params)"
-            transmission_hw_interface="$(arg transmission_hw_interface)"
-            safety_limits="$(arg safety_limits)"
-            safety_pos_margin="$(arg safety_pos_margin)"
-            safety_k_position="$(arg safety_k_position)"
-            use_mock_hardware="$(arg use_mock_hardware)"
-            mock_sensor_commands="$(arg mock_sensor_commands)"
-            robot_ip="$(arg robot_ip)"
-            script_filename="$(arg script_filename)"
-            input_recipe_filename="$(arg input_recipe_filename)"
-            output_recipe_filename="$(arg output_recipe_filename)"
+            parent="${tf_prefix}body_link"
+            name="${name}"
+            tf_prefix="${tf_prefix}"
+            ur_type="${ur_type}"
+            joint_limit_params="${joint_limit_params}"
+            kinematics_params="${kinematics_params}"
+            physical_params="${physical_params}"
+            visual_params="${visual_params}"
+            transmission_hw_interface="${transmission_hw_interface}"
+            safety_limits="${safety_limits}"
+            safety_pos_margin="${safety_pos_margin}"
+            safety_k_position="${safety_k_position}"
+            use_mock_hardware="${use_mock_hardware}"
+            mock_sensor_commands="${mock_sensor_commands}"
+            robot_ip="${robot_ip}"
+            script_filename="${script_filename}"
+            input_recipe_filename="${input_recipe_filename}"
+            output_recipe_filename="${output_recipe_filename}"
             initial_positions="${xacro.load_yaml((initial_positions_file))}"
-            use_gazebo="$(arg use_gazebo)"
-            force_abs_paths="$(arg force_abs_paths)"
+            use_gazebo="${use_gazebo}"
+            force_abs_paths="${force_abs_paths}"
             >
             <origin xyz="0 0 ${caster_offset}" rpy="0 0 0"/>

File: src/devol_moveit_config/config/devol.ros2_control.xacro (robot description, xacro)
@@ -3,5 +3,5 @@
     <xacro:include filename="$(find ur_robot_driver)/urdf/ur.ros2_control.xacro"/>
     <xacro:include filename="$(find robotiq_description)/urdf/robotiq_gripper.ros2_control.xacro"/>
-    <xacro:macro name="devol_ros2_control" params="name prefix use_gazebo:=^|false">
+    <xacro:macro name="devol_ros2_control" params="name tf_prefix use_gazebo:=^|false">
         <ros2_control name="${name}" type="system">
             <hardware>
@@ -15,5 +15,5 @@
                 </xacro:unless>
             </hardware>
-            <joint name="shoulder_pan_joint">
+            <joint name="${tf_prefix}shoulder_pan_joint">
                 <command_interface name="position"/>
                 <state_interface name="position">
@@ -22,5 +22,5 @@
                 <state_interface name="velocity"/>
             </joint>
-            <joint name="shoulder_lift_joint">
+            <joint name="${tf_prefix}shoulder_lift_joint">
                 <command_interface name="position"/>
                 <state_interface name="position">
@@ -29,5 +29,5 @@
                 <state_interface name="velocity"/>
             </joint>
-            <joint name="elbow_joint">
+            <joint name="${tf_prefix}elbow_joint">
                 <command_interface name="position"/>
                 <state_interface name="position">
@@ -36,5 +36,5 @@
                 <state_interface name="velocity"/>
             </joint>
-            <joint name="wrist_1_joint">
+            <joint name="${tf_prefix}wrist_1_joint">
                 <command_interface name="position"/>
                 <state_interface name="position">
@@ -43,5 +43,5 @@
                 <state_interface name="velocity"/>
             </joint>
-            <joint name="wrist_2_joint">
+            <joint name="${tf_prefix}wrist_2_joint">
                 <command_interface name="position"/>
                 <state_interface name="position">
@@ -50,5 +50,5 @@
                 <state_interface name="velocity"/>
             </joint>
-            <joint name="wrist_3_joint">
+            <joint name="${tf_prefix}wrist_3_joint">
                 <command_interface name="position"/>
                 <state_interface name="position">
@@ -57,5 +57,5 @@
                 <state_interface name="velocity"/>
             </joint>
-            <joint name="robotiq_85_left_knuckle_joint">
+            <joint name="${tf_prefix}robotiq_85_left_knuckle_joint">
                 <command_interface name="position"/>
                 <state_interface name="position">
@@ -64,4 +64,9 @@
                 <state_interface name="velocity"/>
             </joint>
+            <joint name="${tf_prefix}robotiq_85_right_knuckle_joint" />
+            <joint name="${tf_prefix}robotiq_85_left_inner_knuckle_joint" />
+            <joint name="${tf_prefix}robotiq_85_right_inner_knuckle_joint" />
+            <joint name="${tf_prefix}robotiq_85_left_finger_tip_joint" />
+            <joint name="${tf_prefix}robotiq_85_right_finger_tip_joint" />
         </ros2_control>
     </xacro:macro>

File: src/devol_moveit_config/config/devol.urdf.xacro (robot description, xacro)
@@ -5,4 +5,4 @@
     <!-- Import control_xacro -->
     <xacro:include filename="$(find devol_moveit_config)/config/devol.ros2_control.xacro" />
-    <xacro:devol_ros2_control prefix="fake" name="FakeSystem"/>
+    <xacro:devol_ros2_control tf_prefix="fake" name="FakeSystem"/>
 </robot>

File: src/diff_drive_description/urdf/diff_drive.gazebo.xacro (robot description, xacro)
@@ -54,4 +54,6 @@
         <left_joint>${tf_prefix}left_wheel_joint</left_joint>
         <right_joint>${tf_prefix}right_wheel_joint</right_joint>
+        <topic>/model/${tf_prefix}devol_drive/cmd_vel</topic>
+        <odom_topic>/model/${tf_prefix}devol_drive/odom</odom_topic>
         <wheel_separation>${wheel_separation}</wheel_separation>
         <wheel_radius>${wheel_radius}</wheel_radius>

File: src/diff_drive_description/urdf/diff_drive.urdf.xacro (robot description, xacro)
@@ -5,4 +5,5 @@
     <xacro:include filename="$(find diff_drive_description)/urdf/diff_drive_macro.urdf.xacro"/>
     <!-- ros2_control description -->
+    <xacro:include filename="$(find diff_drive_description)/urdf/diff_drive.ros2_control.xacro"/>
     <!-- Robot Parameters -->
     <xacro:arg name="parent" default="empty"/>  <!-- Set this to world for rviz and others -->
@@ -18,8 +19,11 @@
     <xacro:arg name="max_linear_acceleration" default="10"/>
     <xacro:arg name="use_gazebo" default="true"/>
+    <xacro:arg name="tf_prefix" default=""/>
     <xacro:property name="body_width" value="$(arg body_width)"/>
     <xacro:property name="wheel_width" value="$(arg wheel_width)"/>
     <xacro:property name="wheel_separation" value="${(body_width) + (wheel_width)}"/>
+    <link name="$(arg parent)"/>
     <xacro:diff_drive
+        tf_prefix="$(arg tf_prefix)"
         parent="$(arg parent)"
         body_length="$(arg body_length)"
@@ -42,3 +46,4 @@
             tf_prefix="$(arg tf_prefix)"/>
     </xacro:if>
+    <xacro:diff_drive_ros2_control name="diff_drive_ros2_control" tf_prefix="$(arg tf_prefix)" use_gazebo="$(arg use_gazebo)"/>
 </robot>

File: src/diff_drive_description/urdf/diff_drive_macro.urdf.xacro (robot description, xacro)
@@ -34,5 +34,4 @@
         <xacro:property name="caster_inertia_z" value="${2.0/5.0 * caster_mass * caster_radius * caster_radius}"/>
         <!-- Body Link -->
-        <link name="${parent}"/>
         <link name="${tf_prefix}body_link">
             <visual>
