Commit message: Tested a little. Manipulator integration still needs some work but I am going to do that in a private repo. This is the minimum to reproduce my final project for Introduction to Robotics without infringing on the professor's answers in a meaningful way.

File: src/devol_description/urdf/devol_macro.urdf.xacro (robot description, xacro)
@@ -46,5 +46,4 @@
             <origin xyz="0 0 0" rpy="0 0 0" />          <!-- position robot in the world -->
         </xacro:ur_robot>
-        <!-- ros2 control instance -->
         <xacro:ur_to_robotiq
             prefix="${tf_prefix}"

File: src/devol_drive_description/urdf/devol_drive.urdf.xacro (robot description, xacro)
@@ -7,5 +7,4 @@
     <xacro:include filename="$(find devol_drive_description)/urdf/devol_drive.ros2_control.xacro"/>
     <!-- Robot Parameters -->
-    <xacro:arg name="parent" default="empty"/>  <!-- Set this to world for rviz and others -->
     <xacro:arg name="name" default="devol_drive"/>
     <xacro:arg name="tf_prefix" default="" />
@@ -25,6 +24,6 @@
     <xacro:arg name="input_recipe_filename" default="None" />
     <xacro:arg name="output_recipe_filename" default="None" />
-    <xacro:arg name="body_length" default="0.5"/>
-    <xacro:arg name="body_width" default="0.3"/>
+    <xacro:arg name="body_length" default="0.4"/>
+    <xacro:arg name="body_width" default="0.25"/>
     <xacro:arg name="body_height" default="0.1"/>
     <xacro:arg name="body_density" default="7850.0"/>
@@ -32,5 +31,5 @@
     <xacro:arg name="wheel_width" default="0.05"/>
     <xacro:arg name="wheel_density" default="900"/>
-    <xacro:arg name="caster_radius" default="0.1"/>
+    <xacro:arg name="caster_radius" default="0.05"/>
     <xacro:arg name="caster_density" default="0.1"/>
     <xacro:arg name="max_linear_acceleration" default="10"/>
@@ -45,5 +44,4 @@
     <xacro:property name="wheel_separation" value="${(body_width) + (wheel_width)}"/>
     <xacro:devol_drive
-        parent="$(arg parent)"
         name="$(arg name)"
         tf_prefix="$(arg tf_prefix)"

File: src/devol_drive_description/urdf/devol_drive_macro.urdf.xacro (robot description, xacro)
@@ -6,5 +6,4 @@
     <xacro:include filename="$(find devol_description)/urdf/devol_macro.urdf.xacro"/>
     <xacro:macro name="devol_drive" params="
-        parent
         name
         tf_prefix
@@ -41,5 +40,4 @@
         <xacro:property name="caster_offset" value="${body_length/2 - caster_radius}"/>
         <xacro:diff_drive
-            parent="${parent}"
             tf_prefix="${tf_prefix}"
             body_length="${body_length}"

File: src/diff_drive_description/urdf/diff_drive.gazebo.xacro (robot description, xacro)
@@ -8,5 +8,5 @@
     <!-- ros_control plugin -->
     <!-- Gazebo Parameters -->
-    <gazebo reference="${tf_prefix}base_link">
+    <gazebo reference="${tf_prefix}body_link">
         <mu1>1.0</mu1>
         <mu2>1.0</mu2>
@@ -70,5 +70,5 @@
         <odom_topic>/odom</odom_topic>
         <frame_id>odom</frame_id>
-        <child_frame_id>${tf_prefix}base_link</child_frame_id>
+        <child_frame_id>${tf_prefix}body_link</child_frame_id>
         <tf_topic>/tf</tf_topic>
       </plugin>

File: src/diff_drive_description/urdf/diff_drive.urdf (robot description, URDF)
Before this commit: robot diff_drive, 5 links, 4 joints
Links:
- removed link diff_drive/base_link
- added link diff_drive/body_link, mass 10; collision box size=0.4 0.25 0.1; visual box size=0.4 0.25 0.1
Joints:
- joint diff_drive/caster_joint: parent diff_drive/base_link -> diff_drive/body_link
- joint diff_drive/left_wheel_joint: parent diff_drive/base_link -> diff_drive/body_link
- joint diff_drive/lidar_joint: parent diff_drive/base_link -> diff_drive/body_link
- joint diff_drive/right_wheel_joint: parent diff_drive/base_link -> diff_drive/body_link

File: src/diff_drive_description/urdf/diff_drive_macro.urdf.xacro (robot description, xacro)
@@ -33,5 +33,5 @@
         <!-- Body Link -->
         <!-- <link name="${tf_prefix}odom" /> -->
-        <link name="${tf_prefix}base_link">
+        <link name="${tf_prefix}body_link">
             <visual>
                 <origin xyz="0.0 0.0 0.0" rpy="0.0 0.0 0.0"/>
@@ -173,10 +173,10 @@
             <origin xyz="0 0 ${wheel_radius+body_height/2}" rpy="0 0 0"/>
             <parent link="${tf_prefix}odom"/>
-            <child link="${tf_prefix}base_link"/>
+            <child link="${tf_prefix}body_link"/>
         </joint> -->
         <!-- Left Wheel Joint -->
         <joint name="${tf_prefix}left_wheel_joint" type="continuous">
             <origin xyz="-${wheel_offset} ${wheel_separation/2} -${wheel_radius/2}" rpy="0 0 0"/>
-            <parent link="${tf_prefix}base_link"/>
+            <parent link="${tf_prefix}body_link"/>
             <child link="${tf_prefix}left_wheel"/>
             <axis xyz="0 1 0"/>
@@ -187,5 +187,5 @@
         <joint name="${tf_prefix}right_wheel_joint" type="continuous">
             <origin xyz="-${wheel_offset} ${-wheel_separation/2} -${wheel_radius/2}" rpy="0 0 0"/>
-            <parent link="${tf_prefix}base_link"/>
+            <parent link="${tf_prefix}body_link"/>
             <child link="${tf_prefix}right_wheel"/>
             <axis xyz="0 1 0"/>
@@ -196,5 +196,5 @@
         <joint name="${tf_prefix}caster_joint" type="fixed">
             <origin xyz="${caster_offset} 0 -${body_height/2+wheel_radius/2}" rpy="0 0 0"/>
-            <parent link="${tf_prefix}base_link"/>
+            <parent link="${tf_prefix}body_link"/>
             <child link="${tf_prefix}caster"/>
         </joint>
@@ -202,5 +202,5 @@
         <joint name="${tf_prefix}lidar_joint" type="fixed">
             <origin xyz="${caster_offset} 0 ${body_height/2+0.02}" rpy="0 0 0"/> <!-- Using the same position as the caster wheel but above it! -->
-            <parent link="${tf_prefix}base_link"/>
+            <parent link="${tf_prefix}body_link"/>
             <child link="${tf_prefix}lidar"/>
         </joint>
