Commit message: Still a work in progress. Need to integrate new changes with existing systems. This change most likely broke everything

File: src/diff_drive_description/urdf/diff_drive.gazebo.xacro (robot description, xacro)
@@ -8,43 +8,51 @@
     <!-- ros_control plugin -->
     <!-- Gazebo Parameters -->
-    <gazebo reference="${tf_prefix}body_link">
+    <gazebo reference="${tf_prefix}base_link">
         <mu1>1.0</mu1>
         <mu2>1.0</mu2>
-        <material>
-            <ambient>0.0 0.0 0.2 1</ambient>
-            <diffuse>0.0 0.0 0.4 1</diffuse>
-            <specular>0.5 0.5 0.7 1</specular>
-            <emissive>0 0 0 1</emissive>
-        </material>
     </gazebo>
-    <gazebo reference="${tf_prefix}right_wheel_link">
+    <gazebo reference="${tf_prefix}right_wheel">
         <mu1>1.0</mu1>
         <mu2>1.0</mu2>
-        <material>
-          <ambient>0.2 0.0 0.2 1</ambient>
-          <diffuse>0.4 0.0 0.4 1</diffuse>
-          <specular>0.5 0.3 0.6 1</specular>
-          <emissive>0 0 0 1</emissive>
-        </material>
     </gazebo>
-    <gazebo reference="${tf_prefix}left_wheel_link">
+    <gazebo reference="${tf_prefix}left_wheel">
         <mu1>1.0</mu1>
         <mu2>1.0</mu2>
-        <material>
-          <ambient>0.2 0.0 0.2 1</ambient>
-          <diffuse>0.4 0.0 0.4 1</diffuse>
-          <specular>0.5 0.3 0.6 1</specular>
-          <emissive>0 0 0 1</emissive>
-        </material>
     </gazebo>
-    <gazebo reference="${tf_prefix}caster_link">
+    <gazebo reference="${tf_prefix}caster">
         <mu1>0.000001</mu1>
         <mu2>0.000001</mu2>
-        <material>
-          <ambient>0.0 0.2 0.0 1</ambient>
-          <diffuse>0.0 0.5 0.0 1</diffuse>
-          <specular>0.4 0.6 0.4 1</specular>
-          <emissive>0 0 0 1</emissive>
-          </material>
+    </gazebo>
+    <gazebo reference="${tf_prefix}lidar">
+        <mu1>1.0</mu1>
+        <mu2>1.0</mu2>
+        <sensor name='lidar_sensor' type='gpu_lidar'>
+          <pose>0 0 0 0 0 0</pose>
+          <topic>/lidar</topic>
+          <update_rate>10</update_rate>
+          <frame_id>diff_drive/lidar</frame_id>
+          <lidar>
+            <scan>
+              <horizontal>
+                <samples>36</samples>
+                <resolution>1</resolution>
+                <min_angle>-3.14159</min_angle>
+                <max_angle>3.14159</max_angle>
+              </horizontal>
+            </scan>
+            <range>
+              <min>0.1</min>
+              <max>30.0</max>
+              <resolution>0.01</resolution>
+            </range>
+            <noise>
+              <type>gaussian</type>
+              <mean>0.0</mean>
+              <stddev>0.01</stddev>
+            </noise>
+          </lidar>
+          <always_on>1</always_on>
+          <visualize>true</visualize>
+        </sensor>
     </gazebo>
     <gazebo>
@@ -54,18 +62,33 @@
         <left_joint>${tf_prefix}left_wheel_joint</left_joint>
         <right_joint>${tf_prefix}right_wheel_joint</right_joint>
-        <topic>/model/${tf_prefix}devol_drive/cmd_vel</topic>
-        <odom_topic>/model/${tf_prefix}devol_drive/odom</odom_topic>
         <wheel_separation>${wheel_separation}</wheel_separation>
         <wheel_radius>${wheel_radius}</wheel_radius>
-        <odom_publish_frequency>1</odom_publish_frequency>
-        <max_linear_acceleration>${max_linear_acceleration}</max_linear_acceleration>
-        <min_linear_acceleration>-1</min_linear_acceleration>
-        <max_angular_acceleration>2</max_angular_acceleration>
-        <min_angular_acceleration>-2</min_angular_acceleration>
-        <max_linear_velocity>0.5</max_linear_velocity>
-        <min_linear_velocity>-0.5</min_linear_velocity>
-        <max_angular_velocity>1</max_angular_velocity>
-        <min_angular_velocity>-1</min_angular_velocity>
+        <odom_publish_frequency>30</odom_publish_frequency>
+        <max_wheel_torque>2.0</max_wheel_torque>
+        <max_wheel_acceleration>0.75</max_wheel_acceleration>
+        <topic>/cmd_vel</topic>
+        <odom_topic>/odom</odom_topic>
+        <frame_id>odom</frame_id>
+        <child_frame_id>${tf_prefix}base_link</child_frame_id>
+        <tf_topic>/tf</tf_topic>
       </plugin>
+       <plugin filename="gz-sim-joint-state-publisher-system" name="gz::sim::systems::JointStatePublisher">
+            <topic>/joint_states</topic>
+            <publish_tf>false</publish_tf>
+       </plugin>
+       <plugin filename="gz-sim-pose-publisher-system" name="gz::sim::systems::PosePublisher">
+           <publish_link_pose>true</publish_link_pose>
+           <publish_sensor_pose>false</publish_sensor_pose>
+           <publish_collision_pose>false</publish_collision_pose>
+           <publish_visual_pose>false</publish_visual_pose>
+           <publish_nested_model_pose>true</publish_nested_model_pose>
+           <use_pose_vector_msg>true</use_pose_vector_msg>
+           <static_publisher>false</static_publisher>
+           <update_frequency>30</update_frequency>
+           <topic>/model/diff_drive/pose</topic>
+       </plugin>
+       <plugin filename="gz-sim-sensors-system" name="gz::sim::systems::Sensors">
+           <render_engine>ogre2</render_engine>
+       </plugin>
     </gazebo>
   </xacro:macro>

File: src/diff_drive_description/urdf/diff_drive.urdf.xacro (robot description, xacro)
@@ -7,7 +7,6 @@
     <xacro:include filename="$(find diff_drive_description)/urdf/diff_drive.ros2_control.xacro"/>
     <!-- Robot Parameters -->
-    <xacro:arg name="parent" default="empty"/>  <!-- Set this to world for rviz and others -->
-    <xacro:arg name="body_length" default="0.5"/>
-    <xacro:arg name="body_width" default="0.3"/>
+    <xacro:arg name="body_length" default="0.4"/>
+    <xacro:arg name="body_width" default="0.25"/>
     <xacro:arg name="body_height" default="0.1"/>
     <xacro:arg name="body_density" default="7850.0"/>
@@ -15,5 +14,5 @@
     <xacro:arg name="wheel_width" default="0.05"/>
     <xacro:arg name="wheel_density" default="900"/>
-    <xacro:arg name="caster_radius" default="0.1"/>
+    <xacro:arg name="caster_radius" default="0.05"/>
     <xacro:arg name="caster_density" default="0.1"/>
     <xacro:arg name="max_linear_acceleration" default="10"/>
@@ -22,9 +21,10 @@
     <xacro:property name="body_width" value="$(arg body_width)"/>
     <xacro:property name="wheel_width" value="$(arg wheel_width)"/>
+    <xacro:property name="body_length" value="$(arg body_length)"/>
+    <xacro:property name="caster_radius" value="$(arg caster_radius)"/>
     <xacro:property name="wheel_separation" value="${(body_width) + (wheel_width)}"/>
-    <link name="$(arg parent)"/>
+    <xacro:property name="caster_offset" value="${(body_length)/2 - (caster_radius)}"/>
     <xacro:diff_drive
         tf_prefix="$(arg tf_prefix)"
-        parent="$(arg parent)"
         body_length="$(arg body_length)"
         body_width="$(arg body_width)"

File: src/diff_drive_description/urdf/diff_drive_macro.urdf.xacro (robot description, xacro)
@@ -1,4 +1,3 @@
 <?xml version="1.0"?>
-<!-- Reference: https://github.com/lucasmazzetto/gazebo_differential_drive_robot -->
 <robot xmlns:xacro="http://wiki.ros.org/xacro">
     <!-- import macros -->
@@ -6,5 +5,4 @@
     <xacro:macro name="diff_drive" params="
         tf_prefix
-        parent:=empty
         body_length:=0.5
         body_width:=0.3
@@ -14,5 +12,5 @@
         wheel_width:=0.05
         wheel_density:=900
-        caster_radius:=0.1
+        caster_radius:=0.05
         caster_density:=0.1
         max_linear_acceleration:=10
@@ -34,5 +32,6 @@
         <xacro:property name="caster_inertia_z" value="${2.0/5.0 * caster_mass * caster_radius * caster_radius}"/>
         <!-- Body Link -->
-        <link name="${tf_prefix}body_link">
+        <!-- <link name="${tf_prefix}odom" /> -->
+        <link name="${tf_prefix}base_link">
             <visual>
                 <origin xyz="0.0 0.0 0.0" rpy="0.0 0.0 0.0"/>
@@ -40,5 +39,5 @@
                     <box size="${body_length} ${body_width} ${body_height}"/>
                 </geometry>
-                <material name="dark-blue-metal" />
+                <material name="chasis-material" />
             </visual>
             <collision>
@@ -54,17 +53,12 @@
             </inertial>
         </link>
-        <joint name="${tf_prefix}base_to_body" type="fixed">
-            <parent link="${parent}"/>
-            <child link="${tf_prefix}body_link"/>
-            <origin xyz="0 0 ${caster_offset}" rpy="0 0 0"/>
-        </joint>
         <!-- Left Wheel -->
-        <link name="${tf_prefix}left_wheel_link">
-            <visual>
-                <origin xyz="0.0 0.0 0.0" rpy="1.570795 0.0 0.0"/>
-                <geometry>
-                    <cylinder radius="${wheel_radius}" length="${wheel_width}"/>
-                </geometry>
-                <material name="dark-purple-metal" />
+        <link name="${tf_prefix}left_wheel">
+            <visual>
+                <origin xyz="0.0 0.0 0.0" rpy="1.570795 0.0 0.0"/>
+                <geometry>
+                    <cylinder radius="${wheel_radius}" length="${wheel_width}"/>
+                </geometry>
+                <material name="left-wheel-material" />
             </visual>
             <collision>
@@ -97,11 +91,11 @@
         </link>
         <!-- Right Wheel -->
-        <link name="${tf_prefix}right_wheel_link">
-            <visual>
-                <origin xyz="0.0 0.0 0.0" rpy="1.570795 0.0 0.0"/>
-                <geometry>
-                    <cylinder radius="${wheel_radius}" length="${wheel_width}"/>
-                </geometry>
-                <material name="dark-purple-metal" />
+        <link name="${tf_prefix}right_wheel">
+            <visual>
+                <origin xyz="0.0 0.0 0.0" rpy="1.570795 0.0 0.0"/>
+                <geometry>
+                    <cylinder radius="${wheel_radius}" length="${wheel_width}"/>
+                </geometry>
+                <material name="right-wheel-material" />
             </visual>
             <collision>
@@ -134,5 +128,5 @@
         </link>
         <!-- Caster Wheel -->
-        <link name="${tf_prefix}caster_link">
+        <link name="${tf_prefix}caster">
             <visual>
                 <origin xyz="0.0 0.0 0.0" rpy="0.0 0.0 0.0"/>
@@ -140,5 +134,5 @@
                     <sphere radius="${caster_radius}"/>
                 </geometry>
-                <material name="metallic-green" />
+                <material name="caster-wheel-material" />
             </visual>
             <collision>
@@ -154,10 +148,36 @@
             </inertial>
         </link>
+        <!-- LIDAR -->
+        <link name="${tf_prefix}lidar">
+            <inertial>
+                <mass value="0.1"/>
+                <inertia ixx="0.0000027" ixy="0.0" ixz="0.0" iyy="0.0000027" iyz="0" izz="0.0000027"/>
+                <origin xyz="0 0 0" rpy="0 0 0"/>
+            </inertial>
+            <visual>
+                <origin xyz="0.0 0.0 0.0" rpy="0.0 0.0 0.0"/>
+                <geometry>
+                    <cylinder radius="0.01" length="0.04"/>
+                </geometry>
+                <material name="lidar-material" />
+            </visual>
+            <collision>
+                <geometry>
+                    <cylinder radius="0.01" length="0.04"/>
+                </geometry>
+            </collision>
+        </link>
         <!-- Joints -->
+        <!-- Floor Joint -->
+        <!-- <joint name="${tf_prefix}floor_fixed_joint" type="fixed">
+            <origin xyz="0 0 ${wheel_radius+body_height/2}" rpy="0 0 0"/>
+            <parent link="${tf_prefix}odom"/>
+            <child link="${tf_prefix}base_link"/>
+        </joint> -->
         <!-- Left Wheel Joint -->
         <joint name="${tf_prefix}left_wheel_joint" type="continuous">
             <origin xyz="-${wheel_offset} ${wheel_separation/2} -${wheel_radius/2}" rpy="0 0 0"/>
-            <parent link="${tf_prefix}body_link"/>
-            <child link="${tf_prefix}left_wheel_link"/>
+            <parent link="${tf_prefix}base_link"/>
+            <child link="${tf_prefix}left_wheel"/>
             <axis xyz="0 1 0"/>
             <limit effort="100" velocity="10.0"/>
@@ -167,15 +187,21 @@
         <joint name="${tf_prefix}right_wheel_joint" type="continuous">
             <origin xyz="-${wheel_offset} ${-wheel_separation/2} -${wheel_radius/2}" rpy="0 0 0"/>
-            <parent link="${tf_prefix}body_link"/>
-            <child link="${tf_prefix}right_wheel_link"/>
+            <parent link="${tf_prefix}base_link"/>
+            <child link="${tf_prefix}right_wheel"/>
             <axis xyz="0 1 0"/>
             <limit effort="100" velocity="10.0"/>
             <dynamics damping="0.1" friction="0.1"/>
         </joint>
-        <!-- Caster Wheel Joint (fixed) -->
+        <!-- Caster Wheel Joint (fixed) or Ball?!? -->
         <joint name="${tf_prefix}caster_joint" type="fixed">
-            <origin xyz="${caster_offset} 0 -${caster_radius/2}" rpy="0 0 0"/>
-            <parent link="${tf_prefix}body_link"/>
-            <child link="${tf_prefix}caster_link"/>
+            <origin xyz="${caster_offset} 0 -${body_height/2+wheel_radius/2}" rpy="0 0 0"/>
+            <parent link="${tf_prefix}base_link"/>
+            <child link="${tf_prefix}caster"/>
+        </joint>
+        <!-- Lidar Joint (fixed) -->
+        <joint name="${tf_prefix}lidar_joint" type="fixed">
+            <origin xyz="${caster_offset} 0 ${body_height/2+0.02}" rpy="0 0 0"/> <!-- Using the same position as the caster wheel but above it! -->
+            <parent link="${tf_prefix}base_link"/>
+            <child link="${tf_prefix}lidar"/>
         </joint>
     </xacro:macro>

File: src/diff_drive_description/urdf/materials.xacro (robot description, xacro)
@@ -1,12 +1,43 @@
 <?xml version="1.0"?>
 <robot xmlns:xacro="http://ros.org/wiki/xacro">
-    <material name="dark-blue-metal">
-        <color rgba="${0/255} ${0/255} ${102/255} 1.0" />
+    <!-- Chasis cool-blue -->
+    <material name="chasis-material">
+        <color rgba="${70/255} ${130/255} ${180/255} 1.0" />
+        <ambient>0.1 0.2 0.3 1</ambient>  <!-- Soft blue under ambient light -->
+        <diffuse>0.3 0.5 0.7 1</diffuse>  <!-- Calm, mid-tone blue under direct lighting -->
+        <specular>0.2 0.3 0.4 1</specular>  <!-- Slight shine with blue undertones -->
+        <emissive>0.0 0.0 0.0 1</emissive>  <!-- No glow -->
     </material>
-    <material name="dark-purple-metal">
-        <color rgba="${102/255} ${0/255} ${102/255} 1.0" />
+    <!-- Right Wheel cool-teal -->
+    <material name="right-wheel-material">
+        <color rgba="${0/255} ${128/255} ${128/255} 1.0" />
+        <ambient>0.1 0.3 0.3 1</ambient>  <!-- Muted teal under ambient light -->
+        <diffuse>0.0 0.5 0.5 1</diffuse>  <!-- Teal under direct lighting -->
+        <specular>0.1 0.3 0.3 1</specular>  <!-- Slight shine with a cool tint -->
+        <emissive>0.0 0.0 0.0 1</emissive>  <!-- No glow -->
     </material>
-    <material name="metallic-green">
-        <color rgba="${0/255} ${128/255} ${0/255} 1.0" />
+    <!-- Left Wheel deep-purple -->
+    <material name="left-wheel-material">
+        <color rgba="${80/255} ${0/255} ${128/255} 1.0" />
+        <ambient>0.2 0.0 0.2 1</ambient>  <!-- Soft deep purple under ambient light -->
+        <diffuse>0.5 0.0 0.6 1</diffuse>  <!-- Deep purple under direct lighting -->
+        <specular>0.3 0.0 0.4 1</specular>  <!-- Glossy with purple tint -->
+        <emissive>0.0 0.0 0.0 1</emissive>  <!-- No glow -->
+    </material>
+    <!-- Caster Wheel cool-green -->
+    <material name="caster-wheel-material">
+        <color rgba="${50/255} ${205/255} ${50/255} 1.0" />
+        <ambient>0.1 0.3 0.1 1</ambient>  <!-- Muted lime green under ambient light -->
+        <diffuse>0.2 0.8 0.2 1</diffuse>  <!-- Bright green under direct lighting -->
+        <specular>0.2 0.4 0.2 1</specular>  <!-- Slight shine with a green tint -->
+        <emissive>0.0 0.0 0.0 1</emissive>  <!-- No glow -->
+    </material>
+    <!-- LIDAR laser-red -->
+    <material name="lidar-material">
+        <color rgba="${200/255} ${0/255} ${0/255} 1.0" />
+        <ambient>0.2 0.0 0.0 1</ambient>  <!-- Dim red under ambient light -->
+        <diffuse>1.0 0.0 0.0 1</diffuse>  <!-- Bright red under direct lighting -->
+        <specular>0.3 0.0 0.0 1</specular>  <!-- Glossy red -->
+        <emissive>0.3 0.0 0.0 1</emissive>  <!-- Glowing red (representing laser-like effect) -->
     </material>
 </robot>
