Commit message: Sensors need some work but robot drives well.

File: src/a200_description/urdf/a200.urdf.xacro (robot description, xacro)
@@ -5,25 +5,3 @@
     <xacro:include filename="$(find a200_description)/urdf/a200_macro.urdf.xacro"/>
     <xacro:a200 />
-    <gazebo>
-        <plugin filename="gz-sim-diff-drive-system" name="gz::sim::systems::DiffDrive">
-            <left_joint>front_left_wheel_joint</left_joint>
-            <left_joint>rear_left_wheel_joint</left_joint>
-            <right_joint>front_right_wheel_joint</right_joint>
-            <right_joint>rear_right_wheel_joint</right_joint>
-            <wheel_separation>0.555</wheel_separation>
-            <wheel_radius>0.1651</wheel_radius>
-            <odom_publish_frequency>30</odom_publish_frequency>
-            <max_wheel_torque>2.0</max_wheel_torque>
-            <max_wheel_acceleration>0.75</max_wheel_acceleration>
-            <topic>/a200_0000/cmd_vel</topic>
-            <odom_topic>/a200_0000/odom</odom_topic>
-            <frame_id>odom</frame_id>
-            <child_frame_id>a200_base_link</child_frame_id>
-            <tf_topic>/model/a200_0000/tf</tf_topic>
-            <publish_odom_tf>true</publish_odom_tf>
-        </plugin>
-        <plugin filename="gz-sim-joint-state-publisher-system" name="gz::sim::systems::JointStatePublisher">
-            <topic>/a200_0000/dynamic_joint_states</topic>
-        </plugin>
-    </gazebo>
 </robot>

File: src/a200_description/urdf/a200_macro.urdf.xacro (robot description, xacro)
@@ -641,5 +641,5 @@
             <visual>
             <!-- the mesh origin is at front plate in between the two infrared camera axes -->
-            <origin rpy="1.5707963267948966 0 1.5707963267948966" xyz="0.0043 -0.0175 0"/>
+            <origin rpy="1.5707963267948966 0 -1.5707963267948966" xyz="-0.02 -0.0175 0"/>
             <geometry>
                 <mesh filename="file:///opt/ros/jazzy/share/realsense2_description/meshes/d435.dae"/>
@@ -681,4 +681,28 @@
             </sensor>
         </gazebo>
+        <gazebo>
+            <plugin filename="gz-sim-diff-drive-system" name="gz::sim::systems::DiffDrive">
+                <left_joint>front_left_wheel_joint</left_joint>
+                <left_joint>rear_left_wheel_joint</left_joint>
+                <right_joint>front_right_wheel_joint</right_joint>
+                <right_joint>rear_right_wheel_joint</right_joint>
+                <wheel_separation>0.555</wheel_separation>
+                <wheel_radius>0.1651</wheel_radius>
+                <odom_publish_frequency>30</odom_publish_frequency>
+                <max_wheel_torque>2.0</max_wheel_torque>
+                <max_wheel_acceleration>0.75</max_wheel_acceleration>
+                <topic>/a200_0000/cmd_vel</topic>
+                <odom_topic>/a200_0000/odom</odom_topic>
+                <frame_id>odom</frame_id>
+                <child_frame_id>a200_base_link</child_frame_id>
+                <tf_topic>/model/a200_0000/tf</tf_topic>
+                <publish_odom_tf>true</publish_odom_tf>
+            </plugin>
+        </gazebo>
+        <gazebo>
+            <plugin filename="gz-sim-joint-state-publisher-system" name="gz::sim::systems::JointStatePublisher">
+                <topic>/a200_0000/dynamic_joint_states</topic>
+            </plugin>
+        </gazebo>
     </xacro:macro>
 </robot>
