Commit message: Working cameras

File: src/a200_description/urdf/a200_macro.urdf.xacro (robot description, xacro)
@@ -633,32 +633,9 @@
         </joint>
         <link name="camera_0_bottom_screw_frame"/>
-        <joint name="camera_0_link_joint" type="fixed">
-            <origin rpy="0 0 0" xyz="0.010600000000000002 0.0175 0.0125"/>
-            <parent link="camera_0_bottom_screw_frame"/>
-            <child link="camera_0_link"/>
-        </joint>
-        <link name="camera_0_link">
-            <visual>
-            <!-- the mesh origin is at front plate in between the two infrared camera axes -->
-            <origin rpy="1.5707963267948966 0 -1.5707963267948966" xyz="-0.02 -0.0175 0"/>
-            <geometry>
-                <mesh filename="file:///opt/ros/jazzy/share/realsense2_description/meshes/d435.dae"/>
-            </geometry>
-            </visual>
-            <collision>
-            <origin rpy="0 0 0" xyz="0 -0.0175 0"/>
-            <geometry>
-                <box size="0.02505 0.09 0.025"/>
-            </geometry>
-            </collision>
-            <inertial>
-            <!-- The following are not reliable values, and should not be used for modeling -->
-            <mass value="0.072"/>
-            <origin xyz="0 0 0"/>
-            <inertia ixx="0.003881243" ixy="0.0" ixz="0.0" iyy="0.000498940" iyz="0.0" izz="0.003879257"/>
-            </inertial>
-        </link>
-        <gazebo reference="camera_0_link">
-            <sensor name="camera_0" type="rgbd_camera">
+        <xacro:sensor_d435 parent="camera_0_bottom_screw_frame" name="rear_camera" use_nominal_extrinsics="true">
+            <origin rpy="3.14159 0 3.14159" xyz="0 0 0.022"/>
+        </xacro:sensor_d435>
+        <gazebo reference="rear_camera_color_frame">
+            <sensor name="realsense_d435_camera" type="rgbd_camera">
                 <camera>
                     <horizontal_fov>1.25</horizontal_fov>
@@ -671,11 +648,11 @@
                     <far>100</far>
                     </clip>
-                    <gz_frame_id>camera_0_link</gz_frame_id>
-                    <optical_frame_id>camera_0_color_optical_frame</optical_frame_id>
+                    <gz_frame_id>rear_camera_color_frame</gz_frame_id>
+                    <optical_frame_id>rear_camera_color_frame</optical_frame_id>
                 </camera>
                 <always_on>1</always_on>
                 <update_rate>30</update_rate>
                 <visualize>true</visualize>
-                <gz_frame_id>camera_0_link</gz_frame_id>
+                <gz_frame_id>rear_camera_color_frame</gz_frame_id>
                 <topic>a200_0000/sensors/camera_0</topic>
             </sensor>

File: src/devol_description/urdf/devol.gazebo.xacro (robot description, xacro)
@@ -26,7 +26,7 @@
       <sensor type="camera" name="${tf_prefix}realsense_d405_camera">
         <pose relative_to="${tf_prefix}_camera_color_frame">0 0 0 3.14159 0 0</pose>
-        <topic>/model/${tf_prefix}devol/color_raw</topic>
+        <topic>/${tf_prefix}devol/sensors/camera/image</topic>
         <camera>
-          <camera_info_topic>/model/${tf_prefix}devol/color_info</camera_info_topic>
+          <camera_info_topic>/${tf_prefix}devol/sensors/camera/color_info</camera_info_topic>
           <horizontal_fov>1.518</horizontal_fov>
           <image>
@@ -48,8 +48,8 @@
     <gazebo reference="${tf_prefix}_camera_depth_frame">
       <sensor type="depth_camera" name="${tf_prefix}realsense_d405_depth_camera">
-        <topic>/model/${tf_prefix}devol/depth_raw</topic>
+        <topic>/${tf_prefix}devol/sensors/camera/depth_image</topic>
         <pose relative_to="${tf_prefix}_camera_color_frame">0 0 0 3.14159 0 0</pose>
         <camera>
-          <camera_info_topic>/model/${tf_prefix}devol/depth_info</camera_info_topic>
+          <camera_info_topic>/${tf_prefix}devol/sensors/camera/depth_info</camera_info_topic>
           <horizontal_fov>1.518</horizontal_fov>
           <image>
