Commit message: Tested full sim

File: src/a200_description/urdf/a200.gazebo.xacro (robot description, xacro)
@@ -5,5 +5,5 @@
 -->
 <robot xmlns:xacro="http://ros.org/wiki/xacro">
-    <xacro:macro name="a200_gazebo">
+    <xacro:macro name="a200_gazebo" params="namespace:=/a200_0000" >
         <gazebo>
             <plugin filename="libgz-sim-wheel-slip-system.so" name="gz::sim::systems::WheelSlip">
@@ -60,5 +60,5 @@
             <always_on>true</always_on>
             <gz_frame_id>lidar2d_0_laser</gz_frame_id>
-            <topic>a200_0000/sensors/lidar2d_0/scan</topic>
+            <topic>${namespace}/sensors/lidar2d_0/scan</topic>
             <lidar>
                 <scan>
@@ -90,5 +90,5 @@
             <always_on>true</always_on>
             <gz_frame_id>lidar3d_0_laser</gz_frame_id>
-            <topic>a200_0000/sensors/lidar3d_0/scan</topic>
+            <topic>${namespace}/sensors/lidar3d_0/scan</topic>
             <lidar>
                 <scan>
@@ -133,5 +133,5 @@
                 <visualize>true</visualize>
                 <gz_frame_id>rear_camera_color_frame</gz_frame_id>
-                <topic>a200_0000/sensors/camera_0</topic>
+                <topic>${namespace}/sensors/camera_0</topic>
             </sensor>
         </gazebo>

File: src/a200_description/urdf/a200_macro.urdf.xacro (robot description, xacro)
@@ -5,5 +5,5 @@
     <xacro:include filename="$(find a200_description)/urdf/a200.gazebo.xacro"/>
     <xacro:include filename= "$(find realsense2_description)/urdf/_d435.urdf.xacro"/>
-    <xacro:macro name="a200" >
+    <xacro:macro name="a200" params="namespace:=/a200_0000" >
         <!-- Base link is the center of the robot's bottom plate -->
         <link name="a200_base_link">
@@ -512,5 +512,5 @@
             <origin rpy="3.14159 0 3.14159" xyz="0 0 0.022"/>
         </xacro:sensor_d435>
-        <xacro:a200_gazebo />
+        <xacro:a200_gazebo namespace="${namespace}"/>
     </xacro:macro>
 </robot>

File: src/devol_description/urdf/devol.gazebo.xacro (robot description, xacro)
@@ -5,12 +5,11 @@
 -->
 <robot xmlns:xacro="http://ros.org/wiki/xacro">
-  <xacro:macro name="devol_gazebo" params="tf_prefix">
+  <xacro:macro name="devol_gazebo" params="tf_prefix namespace:=/devol">
     <!-- Camera -->
     <gazebo reference="${tf_prefix}_camera_color_frame">
-      <sensor type="camera" name="${tf_prefix}realsense_d405_camera">
-        <pose relative_to="${tf_prefix}_camera_color_frame">0 0 0 3.14159 0 0</pose>
-        <topic>/${tf_prefix}devol/sensors/camera/image</topic>
+      <sensor type="rgbd_camera" name="${tf_prefix}realsense_d405_camera">
+        <topic>${namespace}/sensors/camera_1</topic>
+        <gz_frame_id>${tf_prefix}_camera_color_frame</gz_frame_id>
         <camera>
-          <camera_info_topic>/${tf_prefix}devol/sensors/camera/color_info</camera_info_topic>
           <horizontal_fov>1.518</horizontal_fov>
           <image>
@@ -25,28 +24,5 @@
         </camera>
         <always_on>1</always_on>
-        <visualize>1</visualize>
-        <update_rate>30</update_rate>
-      </sensor>
-    </gazebo>
-    <!-- Depth Camera  -->
-    <gazebo reference="${tf_prefix}_camera_depth_frame">
-      <sensor type="depth_camera" name="${tf_prefix}realsense_d405_depth_camera">
-        <topic>/${tf_prefix}devol/sensors/camera/depth_image</topic>
-        <pose relative_to="${tf_prefix}_camera_color_frame">0 0 0 3.14159 0 0</pose>
-        <camera>
-          <camera_info_topic>/${tf_prefix}devol/sensors/camera/depth_info</camera_info_topic>
-          <horizontal_fov>1.518</horizontal_fov>
-          <image>
-            <width>1280</width>
-            <height>720</height>
-            <format>L16</format>
-          </image>
-          <clip>
-            <near>0.1</near>
-            <far>5.0</far>
-          </clip>
-        </camera>
-        <always_on>true</always_on>
-        <visualize>1</visualize>
+        <visualize>true</visualize>
         <update_rate>30</update_rate>
       </sensor>

File: src/devol_description/urdf/devol.urdf.xacro (robot description, xacro)
@@ -19,4 +19,5 @@
   <xacro:arg name="output_recipe_filename" default="None" />
   <xacro:arg name="use_gazebo" default="true" />
+  <xacro:arg name="namespace" default="/devol" />
   <!-- initial position for simulations (Mock Hardware, Gazebo, Ignition) -->
   <xacro:arg name="initial_positions_file" default="$(find devol_description)/config/initial_positions.yaml"/>
@@ -58,4 +59,5 @@
     <xacro:devol_gazebo
       tf_prefix="$(arg tf_prefix)"
+      namespace="$(arg namespace)"
       />
      <gazebo>

File: src/devol_drive_description/urdf/devol_drive.gazebo.xacro (robot description, xacro)
@@ -5,10 +5,9 @@
     wheel_radius
     max_linear_acceleration
-    tf_prefix">
+    tf_prefix
+    namespace:=/devol_drive">
     <!-- Gazebo Parameters -->
     <xacro:include filename="$(find devol_description)/urdf/devol.gazebo.xacro"/>
-    <xacro:devol_gazebo
-      tf_prefix="${tf_prefix}"
-      />
+    <xacro:devol_gazebo tf_prefix="${tf_prefix}" namespace="${namespace}" />
   </xacro:macro>
 </robot>

File: src/devol_drive_description/urdf/devol_drive.urdf.xacro (robot description, xacro)
@@ -36,4 +36,5 @@
     <xacro:arg name="use_gazebo" default="true"/>
     <xacro:arg name="force_abs_paths" default="true"/>
+    <xacro:arg name="namespace" default="/devol_drive"/>
     <!-- initial position for simulations (Mock Hardware, Gazebo, Ignition) -->
     <xacro:arg name="initial_positions_file" default="$(find devol_description)/config/initial_positions.yaml"/>
@@ -43,4 +44,6 @@
     <xacro:property name="wheel_width" value="$(arg wheel_width)"/>
     <xacro:property name="wheel_separation" value="${(body_width) + (wheel_width)}"/>
+    <xacro:property name="name" value="$(arg name)"/>
+    <xacro:property name="namespace" value="$(arg namespace)"/>
     <xacro:devol_drive
         name="$(arg name)"
@@ -73,5 +76,6 @@
         caster_radius="$(arg caster_radius)"
         caster_density="$(arg caster_density)"
-        max_linear_acceleration="$(arg max_linear_acceleration)">
+        max_linear_acceleration="$(arg max_linear_acceleration)"
+        namespace="$(arg namespace)">
         <origin xyz="0 0 0" rpy="0 0 0"/>
     </xacro:devol_drive>
@@ -84,23 +88,24 @@
             max_linear_acceleration="$(arg max_linear_acceleration)"
             tf_prefix="$(arg tf_prefix)"
+            namespace="$(arg namespace)"
              />
         <gazebo>
             <plugin filename="gz_ros2_control-system" name="gz_ros2_control::GazeboSimROS2ControlPlugin">
                 <ros>
-                    <namespace>devol_drive</namespace>
-                    <remapping>~/odom:=devol_drive/odom</remapping>
-                    <remapping>~/cmd_vel:=devol_drive/cmd_vel</remapping>
+                    <namespace>${name}</namespace>
+                    <remapping>~/odom:=${namespace}/odom</remapping>
+                    <remapping>~/cmd_vel:=${namespace}/cmd_vel</remapping>
                     <remapping>/tf:=tf</remapping>
                     <remapping>/tf_static:=tf_static</remapping>
                     <remapping>/diagnostics:=diagnostics</remapping>
-                    <remapping>/dynamic_joint_states:=devol_drive/dynamic_joint_states</remapping>
-                    <remapping>joint_states:=devol_drive/joint_states</remapping>
-                    <remapping>~/reference:=devol_drive/cmd_vel</remapping>
-                    <remapping>~/odometry:=devol_drive/odom</remapping>
+                    <remapping>/dynamic_joint_states:=${namespace}/dynamic_joint_states</remapping>
+                    <remapping>joint_states:=${namespace}/joint_states</remapping>
+                    <remapping>~/reference:=${namespace}/cmd_vel</remapping>
+                    <remapping>~/odometry:=${namespace}/odom</remapping>
                 </ros>
                 <parameters>$(find devol_drive_description)/config/ros2_controllers.yaml</parameters>
             </plugin>
             <plugin filename="gz-sim-joint-state-publisher-system" name="gz::sim::systems::JointStatePublisher">
-                <topic>/devol_drive/dynamic_joint_states</topic>
+                <topic>${namespace}/dynamic_joint_states</topic>
             </plugin>
             <plugin filename="gz-sim-diff-drive-system" name="gz::sim::systems::DiffDrive">
@@ -114,9 +119,9 @@
                 <max_wheel_torque>2.0</max_wheel_torque>
                 <max_wheel_acceleration>0.75</max_wheel_acceleration>
-                <topic>/devol_drive/cmd_vel</topic>
-                <odom_topic>/devol_drive/odom</odom_topic>
+                <topic>${namespace}/cmd_vel</topic>
+                <odom_topic>${namespace}/odom</odom_topic>
                 <frame_id>odom</frame_id>
                 <child_frame_id>a200_base_link</child_frame_id>
-                <tf_topic>/model/devol_drive/tf</tf_topic>
+                <tf_topic>/model/${name}/tf</tf_topic>
                 <publish_odom_tf>true</publish_odom_tf>
             </plugin>

File: src/devol_drive_description/urdf/devol_drive_macro.urdf.xacro (robot description, xacro)
@@ -37,7 +37,8 @@
         caster_density:=0.1
         max_linear_acceleration:=10
+        namespace:=/devol_drive
     ">
         <xacro:property name="caster_offset" value="${body_length/2 - caster_radius}"/>
-        <xacro:a200 />
+        <xacro:a200 namespace="${namespace}" />
         <xacro:devol
             parent="${tf_prefix}top_plate_mount_ur"
@@ -61,6 +62,5 @@
             initial_positions="${xacro.load_yaml((initial_positions_file))}"
             use_gazebo="${use_gazebo}"
-            force_abs_paths="${force_abs_paths}"
-            >
+            force_abs_paths="${force_abs_paths}" >
             <origin xyz="0 0 ${caster_offset}" rpy="0 0 0"/>
         </xacro:devol>
