Commit message: Enable Gazebo wheel slip with a wheel_slip_compliance launch argument
The four WheelSlip plugins all had zero compliance, so the plugin added no
slip. Merge them into one plugin (one entry per wheel) and take the
compliance from the xacro arg wheel_slip_compliance, forwarded by
spawn_entities.launch.py (default 0.5 until the Gazebo sweep picks a value;
the xacro default stays 0.0 for other entry points). Lateral and
longitudinal use the same value because the wheel collisions set no fdir1.

Co-Authored-By: Claude Opus 5.5 (1M context) <noreply@anthropic.com>
Claude-Session: https://claude.ai/code/session_01K1wRWhbSx82aqzmwr24HHU

File: src/a200_description/urdf/a200.gazebo.xacro (robot description, xacro)
@@ -5,43 +5,39 @@
 -->
 <robot xmlns:xacro="http://ros.org/wiki/xacro">
+    <xacro:arg name="wheel_slip_compliance" default="0.0"/>
     <xacro:macro name="a200_gazebo" params="namespace:=/a200_0000" >
+        <!-- Wheel slip. Compliance is unitless: the plugin sets each wheel's contact slip to
+             compliance * (wheel_radius * |spin rate|) / wheel_normal_force, so the slip velocity grows
+             with wheel speed and with the friction force (0 = no slip). Lateral and longitudinal use the
+             same value because the wheel collisions set no fdir1, so the engine's friction directions are
+             not tied to the wheel axes. Set with the xacro arg wheel_slip_compliance (spawn_entities.launch.py
+             forwards the launch argument of the same name). -->
+        <xacro:property name="wheel_slip_compliance" value="$(arg wheel_slip_compliance)"/>
         <gazebo>
             <plugin filename="libgz-sim-wheel-slip-system.so" name="gz::sim::systems::WheelSlip">
-            <wheel link_name="front_left_wheel_link">
-                <slip_compliance_lateral>0.0</slip_compliance_lateral>
-                <slip_compliance_longitudinal>0.0</slip_compliance_longitudinal>
-                <wheel_normal_force>113</wheel_normal_force>
-                <wheel_radius>0.1651</wheel_radius>
-            </wheel>
-            </plugin>
-        </gazebo>
-        <gazebo>
-            <plugin filename="libgz-sim-wheel-slip-system.so" name="gz::sim::systems::WheelSlip">
-            <wheel link_name="front_right_wheel_link">
-                <slip_compliance_lateral>0.0</slip_compliance_lateral>
-                <slip_compliance_longitudinal>0.0</slip_compliance_longitudinal>
-                <wheel_normal_force>113</wheel_normal_force>
-                <wheel_radius>0.1651</wheel_radius>
-            </wheel>
-            </plugin>
-        </gazebo>
-        <gazebo>
-            <plugin filename="libgz-sim-wheel-slip-system.so" name="gz::sim::systems::WheelSlip">
-            <wheel link_name="rear_left_wheel_link">
-                <slip_compliance_lateral>0.0</slip_compliance_lateral>
-                <slip_compliance_longitudinal>0.0</slip_compliance_longitudinal>
-                <wheel_normal_force>113</wheel_normal_force>
-                <wheel_radius>0.1651</wheel_radius>
-            </wheel>
-            </plugin>
-        </gazebo>
-        <gazebo>
-            <plugin filename="libgz-sim-wheel-slip-system.so" name="gz::sim::systems::WheelSlip">
-            <wheel link_name="rear_right_wheel_link">
-                <slip_compliance_lateral>0.0</slip_compliance_lateral>
-                <slip_compliance_longitudinal>0.0</slip_compliance_longitudinal>
-                <wheel_normal_force>113</wheel_normal_force>
-                <wheel_radius>0.1651</wheel_radius>
-            </wheel>
+                <wheel link_name="front_left_wheel_link">
+                    <slip_compliance_lateral>${wheel_slip_compliance}</slip_compliance_lateral>
+                    <slip_compliance_longitudinal>${wheel_slip_compliance}</slip_compliance_longitudinal>
+                    <wheel_normal_force>113</wheel_normal_force>
+                    <wheel_radius>0.1651</wheel_radius>
+                </wheel>
+                <wheel link_name="front_right_wheel_link">
+                    <slip_compliance_lateral>${wheel_slip_compliance}</slip_compliance_lateral>
+                    <slip_compliance_longitudinal>${wheel_slip_compliance}</slip_compliance_longitudinal>
+                    <wheel_normal_force>113</wheel_normal_force>
+                    <wheel_radius>0.1651</wheel_radius>
+                </wheel>
+                <wheel link_name="rear_left_wheel_link">
+                    <slip_compliance_lateral>${wheel_slip_compliance}</slip_compliance_lateral>
+                    <slip_compliance_longitudinal>${wheel_slip_compliance}</slip_compliance_longitudinal>
+                    <wheel_normal_force>113</wheel_normal_force>
+                    <wheel_radius>0.1651</wheel_radius>
+                </wheel>
+                <wheel link_name="rear_right_wheel_link">
+                    <slip_compliance_lateral>${wheel_slip_compliance}</slip_compliance_lateral>
+                    <slip_compliance_longitudinal>${wheel_slip_compliance}</slip_compliance_longitudinal>
+                    <wheel_normal_force>113</wheel_normal_force>
+                    <wheel_radius>0.1651</wheel_radius>
+                </wheel>
             </plugin>
         </gazebo>

Commit message: Port the sim to ROS 2 Lyrical and Gazebo Jetty
devol_gazebo still built against Gazebo Harmonic (gz-cmake3), so main did not
build on Lyrical. These are the fixes the sim has been running with locally:
Jetty vendor packages for devol_gazebo, vendored Clearpath meshes and an
environment hook for a200_description, the TF bridge and map -> odom changes,
MoveIt dropped from spawn_entities, and the camera toggle.

Co-Authored-By: Claude Opus 5.5 (1M context) <noreply@anthropic.com>

File: src/a200_description/urdf/a200.gazebo.xacro (robot description, xacro)
@@ -5,5 +5,5 @@
 -->
 <robot xmlns:xacro="http://ros.org/wiki/xacro">
-    <xacro:macro name="a200_gazebo" params="namespace:=/a200_0000" >
+    <xacro:macro name="a200_gazebo" params="namespace:=/a200_0000 use_cameras:=true" >
         <gazebo>
             <plugin filename="libgz-sim-wheel-slip-system.so" name="gz::sim::systems::WheelSlip">
@@ -69,5 +69,5 @@
         <gazebo reference="lidar2d_0_laser">
             <sensor name="lidar2d_0" type="gpu_lidar">
-            <update_rate>40</update_rate>
+            <update_rate>20</update_rate>
             <visualize>true</visualize>
             <always_on>true</always_on>
@@ -99,5 +99,5 @@
         <gazebo reference="lidar3d_0_laser">
             <sensor name="lidar3d_0" type="gpu_lidar">
-            <update_rate>20</update_rate>
+            <update_rate>10</update_rate>
             <visualize>true</visualize>
             <always_on>true</always_on>
@@ -127,4 +127,5 @@
             </sensor>
         </gazebo>
+        <xacro:if value="${use_cameras}">
         <gazebo reference="rear_camera_color_frame">
             <sensor name="realsense_d435_camera" type="rgbd_camera">
@@ -149,4 +150,5 @@
             </sensor>
         </gazebo>
+        </xacro:if>
     </xacro:macro>
 </robot>

File: src/a200_description/urdf/a200_macro.urdf.xacro (robot description, xacro)
@@ -5,5 +5,5 @@
     <xacro:include filename="$(find a200_description)/urdf/a200.gazebo.xacro"/>
     <xacro:include filename= "$(find realsense2_description)/urdf/_d435.urdf.xacro"/>
-    <xacro:macro name="a200" params="namespace:=/a200_0000" >
+    <xacro:macro name="a200" params="namespace:=/a200_0000 use_cameras:=true" >
         <!-- Base link is the center of the robot's bottom plate -->
         <link name="a200_base_link">
@@ -11,5 +11,5 @@
             <origin rpy="0 0 0" xyz="0 0 0"/>
             <geometry>
-                <mesh filename="file:///opt/ros/jazzy/share/clearpath_platform_description/meshes/a200/base_link.dae"/>
+                <mesh filename="package://a200_description/meshes/clearpath_platform_description/a200/base_link.dae"/>
             </geometry>
             </visual>
@@ -32,5 +32,5 @@
             <origin rpy="0 0 0" xyz="0 0 0"/>
             <geometry>
-                <mesh filename="file:///opt/ros/jazzy/share/clearpath_platform_description/meshes/a200/top_chassis.dae"/>
+                <mesh filename="package://a200_description/meshes/clearpath_platform_description/a200/top_chassis.dae"/>
             </geometry>
             </visual>
@@ -64,5 +64,5 @@
             <origin rpy="0 0 0" xyz="0 0 0"/>
             <geometry>
-                <mesh filename="file:///opt/ros/jazzy/share/clearpath_platform_description/meshes/a200/wheels/outdoor.dae"/>
+                <mesh filename="package://a200_description/meshes/clearpath_platform_description/a200/wheels/outdoor.dae"/>
             </geometry>
             </visual>
@@ -89,5 +89,5 @@
             <origin rpy="0 0 0" xyz="0 0 0"/>
             <geometry>
-                <mesh filename="file:///opt/ros/jazzy/share/clearpath_platform_description/meshes/a200/wheels/outdoor.dae"/>
+                <mesh filename="package://a200_description/meshes/clearpath_platform_description/a200/wheels/outdoor.dae"/>
             </geometry>
             </visual>
@@ -115,5 +115,5 @@
             <origin rpy="0 0 0" xyz="0 0 0"/>
             <geometry>
-                <mesh filename="file:///opt/ros/jazzy/share/clearpath_platform_description/meshes/a200/wheels/outdoor.dae"/>
+                <mesh filename="package://a200_description/meshes/clearpath_platform_description/a200/wheels/outdoor.dae"/>
             </geometry>
             </visual>
@@ -140,5 +140,5 @@
             <origin rpy="0 0 0" xyz="0 0 0"/>
             <geometry>
-                <mesh filename="file:///opt/ros/jazzy/share/clearpath_platform_description/meshes/a200/wheels/outdoor.dae"/>
+                <mesh filename="package://a200_description/meshes/clearpath_platform_description/a200/wheels/outdoor.dae"/>
             </geometry>
             </visual>
@@ -226,5 +226,5 @@
             <visual>
             <geometry>
-                <mesh filename="file:///opt/ros/jazzy/share/clearpath_platform_description/meshes/a200/attachments/bumper.dae"/>
+                <mesh filename="package://a200_description/meshes/clearpath_platform_description/a200/attachments/bumper.dae"/>
             </geometry>
             </visual>
@@ -246,5 +246,5 @@
             <visual>
             <geometry>
-                <mesh filename="file:///opt/ros/jazzy/share/clearpath_platform_description/meshes/a200/attachments/bumper.dae"/>
+                <mesh filename="package://a200_description/meshes/clearpath_platform_description/a200/attachments/bumper.dae"/>
             </geometry>
             </visual>
@@ -269,5 +269,5 @@
             <material name="clearpath_dark_grey"/>
             <geometry>
-                <mesh filename="file:///opt/ros/jazzy/share/clearpath_platform_description/meshes/a200/attachments/pacs_top_plate.stl"/>
+                <mesh filename="package://a200_description/meshes/clearpath_platform_description/a200/attachments/pacs_top_plate.stl"/>
             </geometry>
             </visual>
@@ -308,5 +308,5 @@
             <origin rpy="0 0 0" xyz="0 0 0.3"/>
             <geometry>
-                <mesh filename="file:///opt/ros/jazzy/share/clearpath_platform_description/meshes/a200/attachments/300_mm_sensor_arch.dae"/>
+                <mesh filename="package://a200_description/meshes/clearpath_platform_description/a200/attachments/300_mm_sensor_arch.dae"/>
             </geometry>
             </visual>
@@ -314,5 +314,5 @@
             <origin rpy="0 0 0" xyz="0 0 0.3"/>
             <geometry>
-                <mesh filename="file:///opt/ros/jazzy/share/clearpath_platform_description/meshes/a200/attachments/300_mm_sensor_arch.dae"/>
+                <mesh filename="package://a200_description/meshes/clearpath_platform_description/a200/attachments/300_mm_sensor_arch.dae"/>
             </geometry>
             </collision>
@@ -354,5 +354,5 @@
             <visual>
             <geometry>
-                <mesh filename="file:///opt/ros/jazzy/share/clearpath_mounts_description/meshes/fath_pivot_mount_base.dae"/>
+                <mesh filename="package://a200_description/meshes/clearpath_mounts_description/fath_pivot_mount_base.dae"/>
             </geometry>
             <origin rpy="0 0 1.5707963267948966" xyz="0 0 0"/>
@@ -374,5 +374,5 @@
             <visual>
             <geometry>
-                <mesh filename="file:///opt/ros/jazzy/share/clearpath_mounts_description/meshes/fath_pivot_mount.dae"/>
+                <mesh filename="package://a200_description/meshes/clearpath_mounts_description/fath_pivot_mount.dae"/>
             </geometry>
             <origin rpy="0 0 1.5707963267948966" xyz="0 0 0"/>
@@ -405,5 +405,5 @@
             <material name="clearpath_dark_grey"/>
             <geometry>
-                <mesh filename="file:///opt/ros/jazzy/share/clearpath_mounts_description/meshes/pacs/bracket_horizontal.stl"/>
+                <mesh filename="package://a200_description/meshes/clearpath_mounts_description/pacs/bracket_horizontal.stl"/>
             </geometry>
             <origin rpy="0 0 0" xyz="0 0 0.010125"/>
@@ -433,5 +433,5 @@
             <geometry>
                 <!-- Origin of this mesh is the base of the bracket. -->
-                <mesh filename="file:///opt/ros/jazzy/share/clearpath_sensors_description/meshes/hokuyo_ust.stl"/>
+                <mesh filename="package://a200_description/meshes/clearpath_sensors_description/hokuyo_ust.stl"/>
             </geometry>
             <material name="clearpath_dark_grey"/>
@@ -464,10 +464,10 @@
             <visual>
             <geometry>
-                <mesh filename="file:///opt/ros/jazzy/share/velodyne_description/meshes/VLP16_base_1.dae"/>
-            </geometry>
-            </visual>
-            <visual>
-            <geometry>
-                <mesh filename="file:///opt/ros/jazzy/share/velodyne_description/meshes/VLP16_base_2.dae"/>
+                <mesh filename="package://a200_description/meshes/velodyne_description/VLP16_base_1.dae"/>
+            </geometry>
+            </visual>
+            <visual>
+            <geometry>
+                <mesh filename="package://a200_description/meshes/velodyne_description/VLP16_base_2.dae"/>
             </geometry>
             </visual>
@@ -493,5 +493,5 @@
             <origin xyz="0 0 -0.0377"/>
             <geometry>
-                <mesh filename="file:///opt/ros/jazzy/share/velodyne_description/meshes/VLP16_scan.dae"/>
+                <mesh filename="package://a200_description/meshes/velodyne_description/VLP16_scan.dae"/>
             </geometry>
             </visual>
@@ -512,5 +512,5 @@
             <origin rpy="3.14159 0 3.14159" xyz="0 0 0.022"/>
         </xacro:sensor_d435>
-        <xacro:a200_gazebo namespace="${namespace}"/>
+        <xacro:a200_gazebo namespace="${namespace}" use_cameras="${use_cameras}"/>
     </xacro:macro>
 </robot>

File: src/devol_description/urdf/devol.gazebo.xacro (robot description, xacro)
@@ -5,6 +5,7 @@
 -->
 <robot xmlns:xacro="http://ros.org/wiki/xacro">
-  <xacro:macro name="devol_gazebo" params="tf_prefix namespace:=/devol">
+  <xacro:macro name="devol_gazebo" params="tf_prefix namespace:=/devol use_cameras:=true">
     <!-- Camera -->
+    <xacro:if value="${use_cameras}">
     <gazebo reference="${tf_prefix}_camera_color_frame">
       <sensor type="rgbd_camera" name="${tf_prefix}realsense_d405_camera">
@@ -28,4 +29,5 @@
       </sensor>
     </gazebo>
+    </xacro:if>
   </xacro:macro>
 </robot>

File: src/devol_drive_description/urdf/devol_drive.gazebo.xacro (robot description, xacro)
@@ -6,8 +6,9 @@
     max_linear_acceleration
     tf_prefix
-    namespace:=/devol_drive">
+    namespace:=/devol_drive
+    use_cameras:=true">
     <!-- Gazebo Parameters -->
     <xacro:include filename="$(find devol_description)/urdf/devol.gazebo.xacro"/>
-    <xacro:devol_gazebo tf_prefix="${tf_prefix}" namespace="${namespace}" />
+    <xacro:devol_gazebo tf_prefix="${tf_prefix}" namespace="${namespace}" use_cameras="${use_cameras}" />
   </xacro:macro>
 </robot>

File: src/devol_drive_description/urdf/devol_drive.urdf.xacro (robot description, xacro)
@@ -37,4 +37,5 @@
     <xacro:arg name="force_abs_paths" default="true"/>
     <xacro:arg name="namespace" default="/devol_drive"/>
+    <xacro:arg name="use_cameras" default="true"/>
     <!-- initial position for simulations (Mock Hardware, Gazebo, Ignition) -->
     <xacro:arg name="initial_positions_file" default="$(find devol_description)/config/initial_positions.yaml"/>
@@ -77,5 +78,6 @@
         caster_density="$(arg caster_density)"
         max_linear_acceleration="$(arg max_linear_acceleration)"
-        namespace="$(arg namespace)">
+        namespace="$(arg namespace)"
+        use_cameras="$(arg use_cameras)">
         <origin xyz="0 0 0" rpy="0 0 0"/>
     </xacro:devol_drive>
@@ -89,4 +91,5 @@
             tf_prefix="$(arg tf_prefix)"
             namespace="$(arg namespace)"
+            use_cameras="$(arg use_cameras)"
              />
         <gazebo>
@@ -114,5 +117,7 @@
                 <right_joint>front_right_wheel_joint</right_joint>
                 <right_joint>rear_right_wheel_joint</right_joint>
-                <wheel_separation>0.555</wheel_separation>
+                <!-- Effective skid-steer track width (geometric is 0.555 m). Calibrated in Gazebo so that
+                     odometry yaw matches ground truth for in-place turns; 0.555 over-reported yaw ~2.2x. -->
+                <wheel_separation>1.224</wheel_separation>
                 <wheel_radius>0.1651</wheel_radius>
                 <odom_publish_frequency>30</odom_publish_frequency>

File: src/devol_drive_description/urdf/devol_drive_macro.urdf.xacro (robot description, xacro)
@@ -38,7 +38,8 @@
         max_linear_acceleration:=10
         namespace:=/devol_drive
+        use_cameras:=true
     ">
         <xacro:property name="caster_offset" value="${body_length/2 - caster_radius}"/>
-        <xacro:a200 namespace="${namespace}" />
+        <xacro:a200 namespace="${namespace}" use_cameras="${use_cameras}" />
         <xacro:devol
             parent="${tf_prefix}top_plate_mount_ur"
