Commit message: Consolidate launch files and remove unused code
- devol_sim: fold spawn_entities into motion_planner_sim (planner:=none
  runs the sim and map only); remove full_simulation and world_mapper_sim,
  which were older subsets of it; pack the static point cloud once with
  numpy instead of in a Python loop on every publish (same bytes).
- Description packages: one view.launch.py in devol_drive_description
  shows devol_drive, a200 or devol in RViz (joint sliders) or spawned in
  Gazebo, replacing six view_gz/view_rviz files; one ros_gz_bridge
  launch replaces three; one RViz config replaces three (devol.rviz
  needed the removed MoveIt plugin).
- devol_localization: remove the standalone ekf/pf/hybrid launch files,
  which duplicated localization_stack.launch.py.
- devol_gazebo: remove the template BasicSystem/FullSystem plugins (debug
  logging only), the broken view_world launch and the unused tlt_factory
  world; data-only package now.
- Drop unused xacro args from devol_drive (generated URDF is unchanged),
  stale scripts in bin/, and fix references to removed files.

Co-Authored-By: Claude Opus 5.5 (1M context) <noreply@anthropic.com>
Claude-Session: https://claude.ai/code/session_01E5eDGdrQLBYQCBmASVgUYE

File: src/a200_description/urdf/a200.gazebo.xacro (robot description, xacro)
@@ -11,5 +11,5 @@
              with wheel speed and with the friction force (0 = no slip). Lateral and longitudinal use the
              same value because the wheel collisions set no fdir1, so the engine's friction directions are
-             not tied to the wheel axes. Set with the xacro arg wheel_slip_compliance (spawn_entities.launch.py
+             not tied to the wheel axes. Set with the xacro arg wheel_slip_compliance (devol_sim motion_planner_sim.launch.py
              forwards the launch argument of the same name). -->
         <xacro:property name="wheel_slip_compliance" value="$(arg wheel_slip_compliance)"/>

File: src/devol_drive_description/urdf/devol_drive.gazebo.xacro (robot description, xacro)
@@ -2,7 +2,4 @@
 <robot xmlns:xacro="http://ros.org/wiki/xacro">
   <xacro:macro name="devol_drive_gazebo" params="
-    wheel_separation
-    wheel_radius
-    max_linear_acceleration
     tf_prefix
     namespace:=/devol_drive

File: src/devol_drive_description/urdf/devol_drive.urdf.xacro (robot description, xacro)
@@ -24,14 +24,4 @@
     <xacro:arg name="input_recipe_filename" default="None" />
     <xacro:arg name="output_recipe_filename" default="None" />
-    <xacro:arg name="body_length" default="0.4"/>
-    <xacro:arg name="body_width" default="0.25"/>
-    <xacro:arg name="body_height" default="0.1"/>
-    <xacro:arg name="body_density" default="7850.0"/>
-    <xacro:arg name="wheel_radius" default="0.1"/>
-    <xacro:arg name="wheel_width" default="0.05"/>
-    <xacro:arg name="wheel_density" default="900"/>
-    <xacro:arg name="caster_radius" default="0.05"/>
-    <xacro:arg name="caster_density" default="0.1"/>
-    <xacro:arg name="max_linear_acceleration" default="10"/>
     <xacro:arg name="use_gazebo" default="true"/>
     <xacro:arg name="force_abs_paths" default="true"/>
@@ -42,7 +32,4 @@
     <!-- convert to property to use substitution in function -->
     <xacro:property name="initial_positions_file" default="$(arg initial_positions_file)"/>
-    <xacro:property name="body_width" value="$(arg body_width)"/>
-    <xacro:property name="wheel_width" value="$(arg wheel_width)"/>
-    <xacro:property name="wheel_separation" value="${(body_width) + (wheel_width)}"/>
     <xacro:property name="name" value="$(arg name)"/>
     <xacro:property name="namespace" value="$(arg namespace)"/>
@@ -68,14 +55,4 @@
         use_gazebo="$(arg use_gazebo)"
         force_abs_paths="$(arg use_gazebo)"
-        body_length="$(arg body_length)"
-        body_width="$(arg body_width)"
-        body_height="$(arg body_height)"
-        body_density="$(arg body_density)"
-        wheel_radius="$(arg wheel_radius)"
-        wheel_width="$(arg wheel_width)"
-        wheel_density="$(arg wheel_density)"
-        caster_radius="$(arg caster_radius)"
-        caster_density="$(arg caster_density)"
-        max_linear_acceleration="$(arg max_linear_acceleration)"
         namespace="$(arg namespace)"
         use_cameras="$(arg use_cameras)">
@@ -86,7 +63,4 @@
         <xacro:include filename="$(find devol_drive_description)/urdf/devol_drive.gazebo.xacro"/>
         <xacro:devol_drive_gazebo
-            wheel_separation="${(wheel_separation)}"
-            wheel_radius="$(arg wheel_radius)"
-            max_linear_acceleration="$(arg max_linear_acceleration)"
             tf_prefix="$(arg tf_prefix)"
             namespace="$(arg namespace)"

File: src/devol_drive_description/urdf/devol_drive_macro.urdf.xacro (robot description, xacro)
@@ -27,18 +27,7 @@
         use_gazebo
         force_abs_paths
-        body_length:=0.5
-        body_width:=0.3
-        body_height:=0.1
-        body_density:=7850.0
-        wheel_radius:=0.1
-        wheel_width:=0.05
-        wheel_density:=900
-        caster_radius:=0.1
-        caster_density:=0.1
-        max_linear_acceleration:=10
         namespace:=/devol_drive
         use_cameras:=true
     ">
-        <xacro:property name="caster_offset" value="${body_length/2 - caster_radius}"/>
         <xacro:a200 namespace="${namespace}" use_cameras="${use_cameras}" />
         <xacro:devol
@@ -64,5 +53,5 @@
             use_gazebo="${use_gazebo}"
             force_abs_paths="${force_abs_paths}" >
-            <origin xyz="0 0 ${caster_offset}" rpy="0 0 0"/>
+            <origin xyz="0 0 0.15" rpy="0 0 0"/>
         </xacro:devol>
     </xacro:macro>
